File: LCD.sch (KiCad schematic (older format))
At the start: 27 parts

Commit message: start placement
Parts:
- gave numbers to parts that had none: 27

Commit message: routing
Parts:
- U8: value TXB0102DCT -> NTB0102DP
Changed lines of the file:
@@
 P 4300 6600
 F 0 "U8" H 4300 6011 50  0000 C CNN
-F 1 "TXB0102DCT" H 4550 6150 50  0000 C CNN
+F 1 "NTB0102DP" H 4550 6150 50  0000 C CNN
 F 2 "Package_SO:TSSOP-8_3x3mm_P0.65mm" H 4300 6050 50  0001 C CNN
 F 3 "http://www.ti.com/lit/ds/symlink/txb0102.pdf" H 4300 6570 50  0001 C CNN
