File: AOut.sch (KiCad schematic (older format))
At the start: 19 parts

Commit message: start placement
Parts:
- C71, C72, C73, C74: renamed from C?; footprint (none) -> Capacitor_SMD:C_0603_1608Metric
- R133, R134, R135, R136, R137, R138, R139, R140: renamed from R?; footprint (none) -> Resistor_SMD:R_0603_1608Metric
- U17, U18: renamed from U?; footprint (none) -> Package_SO:SOIC-8_3.9x4.9mm_P1.27mm
- gave numbers to parts that had none: 1
Changed lines of the file:
@@
 $Descr A4 11693 8268
 encoding utf-8
-Sheet 19 19
+Sheet 16 21
 Title ""
 Date ""
@@
 $EndDescr
 $Comp
-L AR2ISS:R R?
+L AR2ISS:R R135
 U 1 1 6073B32B
 P 5400 3550
-F 0 "R?" H 5470 3596 50  0000 L CNN
+F 0 "R135" H 5470 3596 50  0000 L CNN
 F 1 "8.2k" H 5470 3505 50  0000 L CNN
-F 2 "" V 5330 3550 50  0001 C CNN
+F 2 "Resistor_SMD:R_0603_1608Metric" V 5330 3550 50  0001 C CNN
 F 3 "~" H 5400 3550 50  0001 C CNN
 	1    5400 3550
@@
 $EndComp
 $Comp
-L AR2ISS:R R?
+L AR2ISS:R R137
 U 1 1 6073B946
 P 6000 3250
-F 0 "R?" V 5793 3250 50  0000 C CNN
+F 0 "R137" V 5793 3250 50  0000 C CNN
 F 1 "27k" V 5884 3250 50  0000 C CNN
-F 2 "" V 5930 3250 50  0001 C CNN
+F 2 "Resistor_SMD:R_0603_1608Metric" V 5930 3250 50  0001 C CNN
 F 3 "~" H 6000 3250 50  0001 C CNN
 	1    6000 3250
@@
 	6450 2750 6250 2750
 $Comp
-L power:GND #PWR?
+L power:GND #PWR0199
 U 1 1 6073C555
 P 5400 3850
-F 0 "#PWR?" H 5400 3600 50  0001 C CNN
+F 0 "#PWR0199" H 5400 3600 50  0001 C CNN
 F 1 "GND" H 5405 3677 50  0000 C CNN
 F 2 "" H 5400 3850 50  0001 C CNN
@@
 	5400 3850 5400 3700
 $Comp
-L AR2ISS:R R?
+L AR2ISS:R R133
 U 1 1 6073CBD1
 P 4550 2650
-F 0 "R?" V 4343 2650 50  0000 C CNN
+F 0 "R133" V 4343 2650 50  0000 C CNN
 F 1 "1k" V 4434 2650 50  0000 C CNN
-F 2 "" V 4480 2650 50  0001 C CNN
+F 2 "Resistor_SMD:R_0603_1608Metric" V 4480 2650 50  0001 C CNN
 F 3 "~" H 4550 2650 50  0001 C CNN
 	1    4550 2650
@@
 	4000 2650 4400 2650
 $Comp
-L AR2ISS:C C?
+L AR2ISS:C C73
 U 1 1 6073D6CD
 P 4950 3050
-F 0 "C?" H 5065 3096 50  0000 L CNN
+F 0 "C73" H 5065 3096 50  0000 L CNN
 F 1 "100nF" H 5065 3005 50  0000 L CNN
-F 2 "" H 4988 2900 50  0001 C CNN
+F 2 "Capacitor_SMD:C_0603_1608Metric" H 4988 2900 50  0001 C CNN
 F 3 "~" H 4950 3050 50  0001 C CNN
 	1    4950 3050
@@
 	4950 2650 5650 2650
 $Comp
-L power:GND #PWR?
+L power:GND #PWR0197
 U 1 1 6073DBE5
 P 4950 3450
-F 0 "#PWR?" H 4950 3200 50  0001 C CNN
+F 0 "#PWR0197" H 4950 3200 50  0001 C CNN
 F 1 "GND" H 4955 3277 50  0000 C CNN
 F 2 "" H 4950 3450 50  0001 C CNN
@@
 	4950 3450 4950 3200
 $Comp
-L Amplifier_Operational:LM358 U?
+L Amplifier_Operational:LM358 U18
 U 1 1 6073E065
 P 8100 2850
-F 0 "U?" H 8100 3217 50  0000 C CNN
+F 0 "U18" H 8100 3217 50  0000 C CNN
 F 1 "LM358" H 8100 3126 50  0000 C CNN
-F 2 "" H 8100 2850 50  0001 C CNN
+F 2 "Package_SO:SOIC-8_3.9x4.9mm_P1.27mm" H 8100 2850 50  0001 C CNN
 F 3 "http://www.ti.com/lit/ds/symlink/lm2904-n.pdf" H 8100 2850 50  0001 C CNN
 	1    8100 2850
@@
 	8550 2850 8400 2850
 $Comp
-L AR2ISS:R R?
+L AR2ISS:R R139
 U 1 1 6073FEFB
 P 8150 2300
-F 0 "R?" V 7943 2300 50  0000 C CNN
+F 0 "R139" V 7943 2300 50  0000 C CNN
 F 1 "NB" V 8034 2300 50  0000 C CNN
-F 2 "" V 8080 2300 50  0001 C CNN
+F 2 "Resistor_SMD:R_0603_1608Metric" V 8080 2300 50  0001 C CNN
 F 3 "~" H 8150 2300 50  0001 C CNN
 	1    8150 2300
@@
 Connection ~ 8550 2850
 $Comp
-L Connector_Generic:Conn_01x04 J?
+L Connector_Generic:Conn_01x04 J28
 U 1 1 60740DE0
 P 10300 3900
-F 0 "J?" H 10380 3892 50  0000 L CNN
+F 0 "J28" H 10380 3892 50  0000 L CNN
 F 1 "Conn_01x04" H 10380 3801 50  0000 L CNN
 F 2 "" H 10300 3900 50  0001 C CNN
@@
 Connection ~ 8800 2850
 $Comp
-L power:GND #PWR?
+L power:GND #PWR0201
 U 1 1 60741D3E
 P 9950 4400
-F 0 "#PWR?" H 9950 4150 50  0001 C CNN
+F 0 "#PWR0201" H 9950 4150 50  0001 C CNN
 F 1 "GND" H 9955 4227 50  0000 C CNN
 F 2 "" H 9950 4400 50  0001 C CNN
@@
 Connection ~ 9950 4100
 $Comp
-L AR2ISS:R R?
+L AR2ISS:R R136
 U 1 1 60747F92
 P 5400 5750
-F 0 "R?" H 5470 5796 50  0000 L CNN
+F 0 "R136" H 5470 5796 50  0000 L CNN
 F 1 "8.2k" H 5470 5705 50  0000 L CNN
-F 2 "" V 5330 5750 50  0001 C CNN
+F 2 "Resistor_SMD:R_0603_1608Metric" V 5330 5750 50  0001 C CNN
 F 3 "~" H 5400 5750 50  0001 C CNN
 	1    5400 5750
@@
 $EndComp
 $Comp
-L AR2ISS:R R?
+L AR2ISS:R R138
 U 1 1 60747F98
 P 6000 5450
-F 0 "R?" V 5793 5450 50  0000 C CNN
+F 0 "R138" V 5793 5450 50  0000 C CNN
 F 1 "27k" V 5884 5450 50  0000 C CNN
-F 2 "" V 5930 5450 50  0001 C CNN
+F 2 "Resistor_SMD:R_0603_1608Metric" V 5930 5450 50  0001 C CNN
 F 3 "~" H 6000 5450 50  0001 C CNN
 	1    6000 5450
@@
 	6450 4950 6250 4950
 $Comp
-L power:GND #PWR?
+L power:GND #PWR0200
 U 1 1 60747FA6
 P 5400 6050
-F 0 "#PWR?" H 5400 5800 50  0001 C CNN
+F 0 "#PWR0200" H 5400 5800 50  0001 C CNN
 F 1 "GND" H 5405 5877 50  0000 C CNN
 F 2 "" H 5400 6050 50  0001 C CNN
@@
 	5400 6050 5400 5900
 $Comp
-L AR2ISS:R R?
+L AR2ISS:R R134
 U 1 1 60747FAD
 P 4550 4850
-F 0 "R?" V 4343 4850 50  0000 C CNN
+F 0 "R134" V 4343 4850 50  0000 C CNN
 F 1 "1k" V 4434 4850 50  0000 C CNN
-F 2 "" V 4480 4850 50  0001 C CNN
+F 2 "Resistor_SMD:R_0603_1608Metric" V 4480 4850 50  0001 C CNN
 F 3 "~" H 4550 4850 50  0001 C CNN
 	1    4550 4850
@@
 	4000 4850 4400 4850
 $Comp
-L AR2ISS:C C?
+L AR2ISS:C C74
 U 1 1 60747FB6
 P 4950 5250
-F 0 "C?" H 5065 5296 50  0000 L CNN
+F 0 "C74" H 5065 5296 50  0000 L CNN
 F 1 "100nF" H 5065 5205 50  0000 L CNN
-F 2 "" H 4988 5100 50  0001 C CNN
+F 2 "Capacitor_SMD:C_0603_1608Metric" H 4988 5100 50  0001 C CNN
 F 3 "~" H 4950 5250 50  0001 C CNN
 	1    4950 5250
@@
 	4950 4850 5650 4850
 $Comp
-L power:GND #PWR?
+L power:GND #PWR0198
 U 1 1 60747FBF
 P 4950 5650
-F 0 "#PWR?" H 4950 5400 50  0001 C CNN
+F 0 "#PWR0198" H 4950 5400 50  0001 C CNN
 F 1 "GND" H 4955 5477 50  0000 C CNN
 F 2 "" H 4950 5650 50  0001 C CNN
@@
 	8550 5050 8400 5050
 $Comp
-L AR2ISS:R R?
+L AR2ISS:R R140
 U 1 1 60747FD3
 P 8150 4500
-F 0 "R?" V 7943 4500 50  0000 C CNN
+F 0 "R140" V 7943 4500 50  0000 C CNN
 F 1 "NB" V 8034 4500 50  0000 C CNN
-F 2 "" V 8080 4500 50  0001 C CNN
+F 2 "Resistor_SMD:R_0603_1608Metric" V 8080 4500 50  0001 C CNN
 F 3 "~" H 8150 4500 50  0001 C CNN
 	1    8150 4500
@@
 	9500 4000 10100 4000
 $Comp
-L Amplifier_Operational:LM358 U?
+L Amplifier_Operational:LM358 U17
 U 2 1 6074FCAD
 P 5950 4950
-F 0 "U?" H 5950 5317 50  0000 C CNN
+F 0 "U17" H 5950 5317 50  0000 C CNN
 F 1 "LM358" H 5950 5226 50  0000 C CNN
-F 2 "" H 5950 4950 50  0001 C CNN
+F 2 "Package_SO:SOIC-8_3.9x4.9mm_P1.27mm" H 5950 4950 50  0001 C CNN
 F 3 "http://www.ti.com/lit/ds/symlink/lm2904-n.pdf" H 5950 4950 50  0001 C CNN
 	2    5950 4950
@@
 $EndComp
 $Comp
-L Amplifier_Operational:LM358 U?
+L Amplifier_Operational:LM358 U17
 U 3 1 60751767
 P 1600 1750
-F 0 "U?" H 1558 1796 50  0000 L CNN
+F 0 "U17" H 1558 1796 50  0000 L CNN
 F 1 "LM358" H 1558 1705 50  0000 L CNN
-F 2 "" H 1600 1750 50  0001 C CNN
+F 2 "Package_SO:SOIC-8_3.9x4.9mm_P1.27mm" H 1600 1750 50  0001 C CNN
 F 3 "http://www.ti.com/lit/ds/symlink/lm2904-n.pdf" H 1600 1750 50  0001 C CNN
 	3    1600 1750
@@
 $EndComp
 $Comp
-L Amplifier_Operational:LM358 U?
+L Amplifier_Operational:LM358 U18
 U 2 1 60754E0F
 P 8100 5050
-F 0 "U?" H 8100 5417 50  0000 C CNN
+F 0 "U18" H 8100 5417 50  0000 C CNN
 F 1 "LM358" H 8100 5326 50  0000 C CNN
-F 2 "" H 8100 5050 50  0001 C CNN
+F 2 "Package_SO:SOIC-8_3.9x4.9mm_P1.27mm" H 8100 5050 50  0001 C CNN
 F 3 "http://www.ti.com/lit/ds/symlink/lm2904-n.pdf" H 8100 5050 50  0001 C CNN
 	2    8100 5050
@@
 $EndComp
 $Comp
-L Amplifier_Operational:LM358 U?
+L Amplifier_Operational:LM358 U17
 U 1 1 60756DD5
 P 5950 2750
-F 0 "U?" H 5950 3117 50  0000 C CNN
+F 0 "U17" H 5950 3117 50  0000 C CNN
 F 1 "LM358" H 5950 3026 50  0000 C CNN
-F 2 "" H 5950 2750 50  0001 C CNN
+F 2 "Package_SO:SOIC-8_3.9x4.9mm_P1.27mm" H 5950 2750 50  0001 C CNN
 F 3 "http://www.ti.com/lit/ds/symlink/lm2904-n.pdf" H 5950 2750 50  0001 C CNN
 	1    5950 2750
@@
 $EndComp
 $Comp
-L Amplifier_Operational:LM358 U?
+L Amplifier_Operational:LM358 U18
 U 3 1 60758A56
 P 2050 1750
-F 0 "U?" H 2008 1796 50  0000 L CNN
+F 0 "U18" H 2008 1796 50  0000 L CNN
 F 1 "LM358" H 2008 1705 50  0000 L CNN
-F 2 "" H 2050 1750 50  0001 C CNN
+F 2 "Package_SO:SOIC-8_3.9x4.9mm_P1.27mm" H 2050 1750 50  0001 C CNN
 F 3 "http://www.ti.com/lit/ds/symlink/lm2904-n.pdf" H 2050 1750 50  0001 C CNN
 	3    2050 1750
@@
 $EndComp
 $Comp
-L AR2ISS:C C?
+L AR2ISS:C C71
 U 1 1 6075C033
 P 2400 1750
-F 0 "C?" H 2515 1796 50  0000 L CNN
+F 0 "C71" H 2515 1796 50  0000 L CNN
 F 1 "100nF" H 2515 1705 50  0000 L CNN
-F 2 "" H 2438 1600 50  0001 C CNN
+F 2 "Capacitor_SMD:C_0603_1608Metric" H 2438 1600 50  0001 C CNN
 F 3 "~" H 2400 1750 50  0001 C CNN
 	1    2400 1750
@@
 $EndComp
 $Comp
-L AR2ISS:C C?
+L AR2ISS:C C72
 U 1 1 6075C598
 P 2900 1750
-F 0 "C?" H 3015 1796 50  0000 L CNN
+F 0 "C72" H 3015 1796 50  0000 L CNN
 F 1 "100nF" H 3015 1705 50  0000 L CNN
-F 2 "" H 2938 1600 50  0001 C CNN
+F 2 "Capacitor_SMD:C_0603_1608Metric" H 2938 1600 50  0001 C CNN
 F 3 "~" H 2900 1750 50  0001 C CNN
 	1    2900 1750
@@
 $EndComp
 $Comp
-L power:GND #PWR?
+L power:GND #PWR0196
 U 1 1 6076297A
 P 1500 2300
-F 0 "#PWR?" H 1500 2050 50  0001 C CNN
+F 0 "#PWR0196" H 1500 2050 50  0001 C CNN
 F 1 "GND" H 1505 2127 50  0000 C CNN
 F 2 "" H 1500 2300 50  0001 C CNN
@@
 $EndComp
 $Comp
-L power:+12V #PWR?
+L power:+12V #PWR0195
 U 1 1 607639CE
 P 1500 1100
-F 0 "#PWR?" H 1500 950 50  0001 C CNN
+F 0 "#PWR0195" H 1500 950 50  0001 C CNN
 F 1 "+12V" H 1515 1273 50  0000 C CNN
 F 2 "" H 1500 1100 50  0001 C CNN

Commit message: routing
Parts:
- J28: footprint (none) -> AR2ISS:250-204
Changed lines of the file:
@@
 $Descr A4 11693 8268
 encoding utf-8
-Sheet 17 22
+Sheet 15 22
 Title ""
 Date ""
@@
 F 0 "J28" H 10380 3892 50  0000 L CNN
 F 1 "Conn_01x04" H 10380 3801 50  0000 L CNN
-F 2 "" H 10300 3900 50  0001 C CNN
+F 2 "AR2ISS:250-204" H 10300 3900 50  0001 C CNN
 F 3 "~" H 10300 3900 50  0001 C CNN
 	1    10300 3900

Commit message: placement, routing
Connections:
- net at R137.1, R139.2, U17.1: now also U17.5 (+); no longer U18.3 (+)
- net at J28.1 (Pin_1), R139.1: now also U17.6 (-), U17.7; no longer U18.1, U18.2 (-)
- net at R136.1, R138.2: now also U18.2 (-); no longer U17.6 (-)
- net at R138.1, R140.2, U18.5 (+): now also U18.1; no longer U17.7
- net at C74.1, R134.1: now also U18.3 (+); no longer U17.5 (+)
Other:
- moved on the sheet: U17B, U18A
Changed lines of the file:
@@
 $Descr A4 11693 8268
 encoding utf-8
-Sheet 15 22
+Sheet 14 22
 Title ""
 Date ""
@@
 L Amplifier_Operational:LM358 U18
 U 1 1 6073E065
-P 8100 2850
-F 0 "U18" H 8100 3217 50  0000 C CNN
-F 1 "LM358" H 8100 3126 50  0000 C CNN
-F 2 "Package_SO:SOIC-8_3.9x4.9mm_P1.27mm" H 8100 2850 50  0001 C CNN
-F 3 "http://www.ti.com/lit/ds/symlink/lm2904-n.pdf" H 8100 2850 50  0001 C CNN
-	1    8100 2850
+P 5950 4950
+F 0 "U18" H 5950 5317 50  0000 C CNN
+F 1 "LM358" H 5950 5226 50  0000 C CNN
+F 2 "Package_SO:SOIC-8_3.9x4.9mm_P1.27mm" H 5950 4950 50  0001 C CNN
+F 3 "http://www.ti.com/lit/ds/symlink/lm2904-n.pdf" H 5950 4950 50  0001 C CNN
+	1    5950 4950
 	1    0    0    -1
 $EndComp
@@
 L Amplifier_Operational:LM358 U17
 U 2 1 6074FCAD
-P 5950 4950
-F 0 "U17" H 5950 5317 50  0000 C CNN
-F 1 "LM358" H 5950 5226 50  0000 C CNN
-F 2 "Package_SO:SOIC-8_3.9x4.9mm_P1.27mm" H 5950 4950 50  0001 C CNN
-F 3 "http://www.ti.com/lit/ds/symlink/lm2904-n.pdf" H 5950 4950 50  0001 C CNN
-	2    5950 4950
-	1    0    0    -1
-$EndComp
+P 8100 2850
+F 0 "U17" H 8100 3217 50  0000 C CNN
+F 1 "LM358" H 8100 3126 50  0000 C CNN
+F 2 "Package_SO:SOIC-8_3.9x4.9mm_P1.27mm" H 8100 2850 50  0001 C CNN
+F 3 "http://www.ti.com/lit/ds/symlink/lm2904-n.pdf" H 8100 2850 50  0001 C CNN
+	2    8100 2850
+	1    0    0    -1
+$EndComp
