File: SDCard.sch (KiCad schematic (older format))
At the start: 7 parts

Commit message: start placement
Parts:
- C70: renamed from C?; footprint (none) -> Capacitor_SMD:C_0603_1608Metric
- R128, R129, R130, R131, R132: renamed from R?; footprint (none) -> Resistor_SMD:R_0603_1608Metric
- gave numbers to parts that had none: 1
Changed lines of the file:
@@
 $Descr A4 11693 8268
 encoding utf-8
-Sheet 18 19
+Sheet 18 21
 Title ""
 Date ""
@@
 $EndDescr
 $Comp
-L Connector:Micro_SD_Card J?
+L Connector:Micro_SD_Card J27
 U 1 1 60B19F5A
 P 6050 3300
-F 0 "J?" H 6000 4017 50  0000 C CNN
+F 0 "J27" H 6000 4017 50  0000 C CNN
 F 1 "Micro_SD_Card" H 6000 3926 50  0000 C CNN
 F 2 "" H 7200 3600 50  0001 C CNN
@@
 $EndComp
 $Comp
-L AR2ISS:R R?
+L AR2ISS:R R132
 U 1 1 60B1A9A3
 P 4500 2350
-F 0 "R?" H 4570 2396 50  0000 L CNN
+F 0 "R132" H 4570 2396 50  0000 L CNN
 F 1 "47k" H 4570 2305 50  0000 L CNN
-F 2 "" V 4430 2350 50  0001 C CNN
+F 2 "Resistor_SMD:R_0603_1608Metric" V 4430 2350 50  0001 C CNN
 F 3 "~" H 4500 2350 50  0001 C CNN
 	1    4500 2350
@@
 $EndComp
 $Comp
-L AR2ISS:R R?
+L AR2ISS:R R131
 U 1 1 60B1ACDA
 P 4250 2350
-F 0 "R?" H 4320 2396 50  0000 L CNN
+F 0 "R131" H 4320 2396 50  0000 L CNN
 F 1 "47k" H 4320 2305 50  0000 L CNN
-F 2 "" V 4180 2350 50  0001 C CNN
+F 2 "Resistor_SMD:R_0603_1608Metric" V 4180 2350 50  0001 C CNN
 F 3 "~" H 4250 2350 50  0001 C CNN
 	1    4250 2350
@@
 $EndComp
 $Comp
-L AR2ISS:R R?
+L AR2ISS:R R130
 U 1 1 60B1AF67
 P 4000 2350
-F 0 "R?" H 4070 2396 50  0000 L CNN
+F 0 "R130" H 4070 2396 50  0000 L CNN
 F 1 "47k" H 4070 2305 50  0000 L CNN
-F 2 "" V 3930 2350 50  0001 C CNN
+F 2 "Resistor_SMD:R_0603_1608Metric" V 3930 2350 50  0001 C CNN
 F 3 "~" H 4000 2350 50  0001 C CNN
 	1    4000 2350
@@
 $EndComp
 $Comp
-L AR2ISS:R R?
+L AR2ISS:R R129
 U 1 1 60B1B1CC
 P 3750 2350
-F 0 "R?" H 3820 2396 50  0000 L CNN
+F 0 "R129" H 3820 2396 50  0000 L CNN
 F 1 "47k" H 3820 2305 50  0000 L CNN
-F 2 "" V 3680 2350 50  0001 C CNN
+F 2 "Resistor_SMD:R_0603_1608Metric" V 3680 2350 50  0001 C CNN
 F 3 "~" H 3750 2350 50  0001 C CNN
 	1    3750 2350
@@
 $EndComp
 $Comp
-L AR2ISS:R R?
+L AR2ISS:R R128
 U 1 1 60B1B3E6
 P 3500 2350
-F 0 "R?" H 3570 2396 50  0000 L CNN
+F 0 "R128" H 3570 2396 50  0000 L CNN
 F 1 "47k" H 3570 2305 50  0000 L CNN
-F 2 "" V 3430 2350 50  0001 C CNN
+F 2 "Resistor_SMD:R_0603_1608Metric" V 3430 2350 50  0001 C CNN
 F 3 "~" H 3500 2350 50  0001 C CNN
 	1    3500 2350
@@
 $EndComp
 $Comp
-L power:+3V3 #PWR?
+L power:+3V3 #PWR0192
 U 1 1 60B1B7F1
 P 3500 1750
-F 0 "#PWR?" H 3500 1600 50  0001 C CNN
+F 0 "#PWR0192" H 3500 1600 50  0001 C CNN
 F 1 "+3V3" H 3515 1923 50  0000 C CNN
 F 2 "" H 3500 1750 50  0001 C CNN
@@
 	4250 2500 4250 3700
 $Comp
-L power:GND #PWR?
+L power:GND #PWR0193
 U 1 1 60B1F0D1
 P 4800 4050
-F 0 "#PWR?" H 4800 3800 50  0001 C CNN
+F 0 "#PWR0193" H 4800 3800 50  0001 C CNN
 F 1 "GND" H 4805 3877 50  0000 C CNN
 F 2 "" H 4800 4050 50  0001 C CNN
@@
 	4800 3500 5150 3500
 $Comp
-L AR2ISS:C C?
+L AR2ISS:C C70
 U 1 1 60B1FB94
 P 5050 2350
-F 0 "C?" H 5165 2396 50  0000 L CNN
+F 0 "C70" H 5165 2396 50  0000 L CNN
 F 1 "100nF" H 5165 2305 50  0000 L CNN
-F 2 "" H 5088 2200 50  0001 C CNN
+F 2 "Capacitor_SMD:C_0603_1608Metric" H 5088 2200 50  0001 C CNN
 F 3 "~" H 5050 2350 50  0001 C CNN
 	1    5050 2350
@@
 Connection ~ 4800 2000
 $Comp
-L power:GND #PWR?
+L power:GND #PWR0194
 U 1 1 60B20AF9
 P 5050 2600
-F 0 "#PWR?" H 5050 2350 50  0001 C CNN
+F 0 "#PWR0194" H 5050 2350 50  0001 C CNN
 F 1 "GND" H 5055 2427 50  0000 C CNN
 F 2 "" H 5050 2600 50  0001 C CNN

Commit message: add TLE5602
Connections:
- net #CS renamed #CD
- net MISO renamed D0
- net MOSI renamed CMD
- net SCK renamed CLK
Changed lines of the file:
@@
 $Descr A4 11693 8268
 encoding utf-8
-Sheet 16 22
+Sheet 15 22
 Title ""
 Date ""
@@
 	4500 3000 4500 2500
 Text HLabel 3100 3100 0    50   Input ~ 0
-#CS
+#CD
 Text HLabel 3100 3200 0    50   Input ~ 0
-MOSI
+CMD
 Wire Wire Line
 	5150 3300 4800 3300
@@
 	4500 2000 4250 2000
 Text HLabel 3100 3400 0    50   Input ~ 0
-SCK
+CLK
 Wire Wire Line
 	3100 3400 5150 3400
 Text HLabel 3100 3600 0    50   Input ~ 0
-MISO
+D0
 Wire Wire Line
 	3100 3600 3500 3600

Commit message: placement, routing
Parts:
- J27: footprint (none) -> Connector_Card:microSD_HC_Wuerth_693072010801
Changed lines of the file:
@@
 $Descr A4 11693 8268
 encoding utf-8
-Sheet 14 22
+Sheet 13 22
 Title ""
 Date ""
@@
 F 0 "J27" H 6000 4017 50  0000 C CNN
 F 1 "Micro_SD_Card" H 6000 3926 50  0000 C CNN
-F 2 "" H 7200 3600 50  0001 C CNN
+F 2 "Connector_Card:microSD_HC_Wuerth_693072010801" H 7200 3600 50  0001 C CNN
 F 3 "http://katalog.we-online.de/em/datasheet/693072010801.pdf" H 6050 3300 50  0001 C CNN
 	1    6050 3300
