File: MESAOut.sch (KiCad schematic (older format))
At the start: 18 parts

Commit message: start placement
Parts:
- C63, C64, C65, C66: renamed from C?; footprint (none) -> Capacitor_SMD:C_0603_1608Metric
- R111, R112, R113, R114, R115, R116, R117, R118, R119, R120: renamed from R?; footprint (none) -> Resistor_SMD:R_0603_1608Metric
- U14, U15: renamed from U?; footprint (none) -> Package_SO:SOIC-28W_7.5x17.9mm_P1.27mm
- gave numbers to parts that had none: 2

Commit message: placement
Parts:
- J22, J23: footprint (none) -> AR2ISS:250-208
Changed lines of the file:
@@
 $Descr A4 11693 8268
 encoding utf-8
-Sheet 14 21
+Sheet 12 22
 Title ""
 Date ""
@@
 F 0 "J22" H 9580 2192 50  0000 L CNN
 F 1 "Conn_01x08" H 9580 2101 50  0000 L CNN
-F 2 "" H 9500 2200 50  0001 C CNN
+F 2 "AR2ISS:250-208" H 9500 2200 50  0001 C CNN
 F 3 "~" H 9500 2200 50  0001 C CNN
 	1    9500 2200
@@
 F 0 "J23" H 9630 4992 50  0000 L CNN
 F 1 "Conn_01x08" H 9630 4901 50  0000 L CNN
-F 2 "" H 9550 5000 50  0001 C CNN
+F 2 "AR2ISS:250-208" H 9550 5000 50  0001 C CNN
 F 3 "~" H 9550 5000 50  0001 C CNN
 	1    9550 5000

Commit message: add TLE5602
Parts:
- removed U14, U15: NCV7608, Package_SO:SOIC-28W_7.5x17.9mm_P1.27mm, symbol AR2ISS:NCV7608
- added F2: PFRA 050, Fuse:Fuse_BelFuse_0ZRE0005FF_L8.3mm_W3.8mm, symbol Device:Polyfuse
- added U14, U15: TLE75602-ESH, AR2ISS:Infineon_PG-TSDSO-24-21, symbol AR2ISS:TLE75602-ESH
Connections:
- net #CS1: now also U14.1 (CSN)
- net #CS2: now also U15.1 (CSN)
- net +12V: now also F2.2; no longer C65.1, J22.7 (Pin_7), J23.7 (Pin_7)
- net +3V3: now also U14.24 (VDD), U15.24 (VDD)
- net EN1: now also U14.21 (IDLE)
- net EN2: now also U15.21 (IDLE)
- net GND: now also U14.25 (PAD), U14.5 (GND), U15.25 (PAD), U15.5 (GND); no longer J22.8 (Pin_8), J23.8 (Pin_8)
- net PWM_DOUT0: now also U14.23 (IN0)
- net PWM_DOUT1: now also U14.22 (IN1)
- net PWM_DOUT2: now also U15.23 (IN0)
- net PWM_DOUT3: now also U15.22 (IN1)
- net at J22.5 (Pin_5): now also U14.11 (OUT6_S)
- net at J22.6 (Pin_6): now also U14.14 (OUT7_S)
- net at J22.2 (Pin_2): now also U14.17 (OUT3_S)
- net at J22.4 (Pin_4): now also U14.15 (OUT5_S)
- net at J22.3 (Pin_3): now also U14.10 (OUT4_S)
- net at J22.1 (Pin_1): now also U14.8 (OUT2_S)
- net at R113.1: now also U14.2 (SCLK)
- net at R114.1: now also U14.3 (SI)
- net at R115.1: now also U14.4 (SO)
- net at J23.5 (Pin_5): now also U15.11 (OUT6_S)
- net at J23.6 (Pin_6): now also U15.14 (OUT7_S)
- net at J23.2 (Pin_2): now also U15.17 (OUT3_S)
- net at J23.4 (Pin_4): now also U15.15 (OUT5_S)
- net at J23.3 (Pin_3): now also U15.10 (OUT4_S)
- net at J23.1 (Pin_1): now also U15.8 (OUT2_S)
- net at R117.1: now also U15.2 (SCLK)
- net at R118.1: now also U15.3 (SI)
- net at R119.1: now also U15.4 (SO)
- new net: J22.7 (Pin_7), U14.6 (OUT0_LS)
- new net: J22.8 (Pin_8), U14.19 (OUT1_LS)
- new net: J23.7 (Pin_7), U15.6 (OUT0_LS)
- new net: J23.8 (Pin_8), U15.19 (OUT1_LS)
- new net +12VA: C65.1, F2.1, U14.12 (OUT6_D), U14.13 (OUT7_D), U14.16 (OUT5_D), U14.18 (OUT3_D), U14.20 (VS), U14.7 (OUT2_D), U14.9 (OUT4_D), U15.12 (OUT6_D), U15.13 (OUT7_D), U15.16 (OUT5_D), U15.18 (OUT3_D), U15.20 (VS), U15.7 (OUT2_D), U15.9 (OUT4_D)
Other:
- moved on the sheet: C63, C64, C65, C66

Commit message: routing
Parts:
- R111, R112, R116, R120: value 100k -> NB
Changed lines of the file:
@@
 P 6600 2250
 F 0 "R116" V 6550 2050 50  0000 C CNN
-F 1 "100k" V 6550 2450 50  0000 C CNN
+F 1 "NB" V 6550 2450 50  0000 C CNN
 F 2 "Resistor_SMD:R_0603_1608Metric" V 6530 2250 50  0001 C CNN
 F 3 "~" H 6600 2250 50  0001 C CNN
@@
 P 6350 1450
 F 0 "R111" H 6420 1496 50  0000 L CNN
-F 1 "100k" H 6420 1405 50  0000 L CNN
+F 1 "NB" H 6420 1405 50  0000 L CNN
 F 2 "Resistor_SMD:R_0603_1608Metric" V 6280 1450 50  0001 C CNN
 F 3 "~" H 6350 1450 50  0001 C CNN
@@
 P 6650 5050
 F 0 "R120" V 6600 4850 50  0000 C CNN
-F 1 "100k" V 6600 5250 50  0000 C CNN
+F 1 "NB" V 6600 5250 50  0000 C CNN
 F 2 "Resistor_SMD:R_0603_1608Metric" V 6580 5050 50  0001 C CNN
 F 3 "~" H 6650 5050 50  0001 C CNN
@@
 P 6400 4250
 F 0 "R112" H 6470 4296 50  0000 L CNN
-F 1 "100k" H 6470 4205 50  0000 L CNN
+F 1 "NB" H 6470 4205 50  0000 L CNN
 F 2 "Resistor_SMD:R_0603_1608Metric" V 6330 4250 50  0001 C CNN
 F 3 "~" H 6400 4250 50  0001 C CNN

Commit message: ready for jlc
Parts:
- removed C63: 100nF, Capacitor_SMD:C_0603_1608Metric, symbol AR2ISS:C
Changed lines of the file:
@@
 $Descr A4 11693 8268
 encoding utf-8
-Sheet 11 22
+Sheet 10 22
 Title ""
 Date ""
@@
 	7000 1450 7000 1200
 $Comp
-L power:+3V3 #PWR0147
-U 1 1 607C08A4
-P 1000 2250
-F 0 "#PWR0147" H 1000 2100 50  0001 C CNN
-F 1 "+3V3" H 1015 2423 50  0000 C CNN
-F 2 "" H 1000 2250 50  0001 C CNN
-F 3 "" H 1000 2250 50  0001 C CNN
-	1    1000 2250
-	1    0    0    -1
-$EndComp
-$Comp
-L AR2ISS:C C63
-U 1 1 607C0E9D
-P 1000 2550
-F 0 "C63" H 1115 2596 50  0000 L CNN
-F 1 "100nF" H 1115 2505 50  0000 L CNN
-F 2 "Capacitor_SMD:C_0603_1608Metric" H 1038 2400 50  0001 C CNN
-F 3 "~" H 1000 2550 50  0001 C CNN
-	1    1000 2550
-	1    0    0    -1
-$EndComp
-$Comp
 L AR2ISS:C C65
 U 1 1 607C1999
@@
 Wire Wire Line
 	2000 2250 2000 2400
-Wire Wire Line
-	1000 2250 1000 2400
-$Comp
-L power:GND #PWR0148
-U 1 1 607C2CAE
-P 1000 2950
-F 0 "#PWR0148" H 1000 2700 50  0001 C CNN
-F 1 "GND" H 1005 2777 50  0000 C CNN
-F 2 "" H 1000 2950 50  0001 C CNN
-F 3 "" H 1000 2950 50  0001 C CNN
-	1    1000 2950
-	1    0    0    -1
-$EndComp
 $Comp
 L power:GND #PWR0152
@@
 	2000 2950 2000 2700
 Wire Wire Line
-	1000 2700 1000 2950
-Wire Wire Line
 	6750 1200 6750 1550
