File: RS232.sch (KiCad schematic (older format))
At the start: 9 parts

Commit message: start placement
Parts:
- C10, C11, C12, C13, C9: renamed from C?; footprint (none) -> Capacitor_SMD:C_0603_1608Metric
- U1: renamed from U?; footprint (none) -> Package_SO:TSSOP-16_4.4x5mm_P0.65mm
- gave numbers to parts that had none: 3
Changed lines of the file:
@@
 $Descr A4 11693 8268
 encoding utf-8
-Sheet 4 19
+Sheet 4 21
 Title ""
 Date ""
@@
 $EndDescr
 $Comp
-L Interface_UART:MAX3232 U?
+L Interface_UART:MAX3232 U1
 U 1 1 6089B57B
 P 4450 3350
-F 0 "U?" H 4850 4400 50  0000 C CNN
+F 0 "U1" H 4850 4400 50  0000 C CNN
 F 1 "MAX3232" H 4000 4400 50  0000 C CNN
-F 2 "" H 4500 2300 50  0001 L CNN
+F 2 "Package_SO:TSSOP-16_4.4x5mm_P0.65mm" H 4500 2300 50  0001 L CNN
 F 3 "https://datasheets.maximintegrated.com/en/ds/MAX3222-MAX3241.pdf" H 4450 3450 50  0001 C CNN
 	1    4450 3350
@@
 $EndComp
 $Comp
-L AR2ISS:C C?
+L AR2ISS:C C9
 U 1 1 6089CA0B
 P 3300 2600
-F 0 "C?" H 3415 2646 50  0000 L CNN
+F 0 "C9" H 3415 2646 50  0000 L CNN
 F 1 "100n" H 3415 2555 50  0000 L CNN
-F 2 "" H 3338 2450 50  0001 C CNN
+F 2 "Capacitor_SMD:C_0603_1608Metric" H 3338 2450 50  0001 C CNN
 F 3 "~" H 3300 2600 50  0001 C CNN
 	1    3300 2600
@@
 $EndComp
 $Comp
-L AR2ISS:C C?
+L AR2ISS:C C11
 U 1 1 6089D053
 P 5650 2600
-F 0 "C?" H 5765 2646 50  0000 L CNN
+F 0 "C11" H 5765 2646 50  0000 L CNN
 F 1 "100n" H 5765 2555 50  0000 L CNN
-F 2 "" H 5688 2450 50  0001 C CNN
+F 2 "Capacitor_SMD:C_0603_1608Metric" H 5688 2450 50  0001 C CNN
 F 3 "~" H 5650 2600 50  0001 C CNN
 	1    5650 2600
@@
 	5550 3250 5250 3250
 $Comp
-L AR2ISS:C C?
+L AR2ISS:C C13
 U 1 1 6089D4DE
 P 5900 2950
-F 0 "C?" V 5648 2950 50  0000 C CNN
+F 0 "C13" V 5648 2950 50  0000 C CNN
 F 1 "100n" V 5739 2950 50  0000 C CNN
-F 2 "" H 5938 2800 50  0001 C CNN
+F 2 "Capacitor_SMD:C_0603_1608Metric" H 5938 2800 50  0001 C CNN
 F 3 "~" H 5900 2950 50  0001 C CNN
 	1    5900 2950
@@
 $EndComp
 $Comp
-L AR2ISS:C C?
+L AR2ISS:C C12
 U 1 1 6089D692
 P 5700 3250
-F 0 "C?" V 5448 3250 50  0000 C CNN
+F 0 "C12" V 5448 3250 50  0000 C CNN
 F 1 "100n" V 5539 3250 50  0000 C CNN
-F 2 "" H 5738 3100 50  0001 C CNN
+F 2 "Capacitor_SMD:C_0603_1608Metric" H 5738 3100 50  0001 C CNN
 F 3 "~" H 5700 3250 50  0001 C CNN
 	1    5700 3250
@@
 $EndComp
 $Comp
-L power:GND #PWR?
+L power:GND #PWR040
 U 1 1 608A2668
 P 6250 2950
-F 0 "#PWR?" H 6250 2700 50  0001 C CNN
+F 0 "#PWR040" H 6250 2700 50  0001 C CNN
 F 1 "GND" V 6255 2822 50  0000 R CNN
 F 2 "" H 6250 2950 50  0001 C CNN
@@
 $EndComp
 $Comp
-L power:GND #PWR?
+L power:GND #PWR039
 U 1 1 608A297B
 P 6100 3250
-F 0 "#PWR?" H 6100 3000 50  0001 C CNN
+F 0 "#PWR039" H 6100 3000 50  0001 C CNN
 F 1 "GND" V 6105 3122 50  0000 R CNN
 F 2 "" H 6100 3250 50  0001 C CNN
@@
 	6100 3250 5850 3250
 $Comp
-L power:GND #PWR?
+L power:GND #PWR037
 U 1 1 609F24C7
 P 4450 4700
-F 0 "#PWR?" H 4450 4450 50  0001 C CNN
+F 0 "#PWR037" H 4450 4450 50  0001 C CNN
 F 1 "GND" H 4455 4527 50  0000 C CNN
 F 2 "" H 4450 4700 50  0001 C CNN
@@
 	4450 4700 4450 4550
 $Comp
-L power:+3V3 #PWR?
+L power:+3V3 #PWR036
 U 1 1 609F715F
 P 4450 1450
-F 0 "#PWR?" H 4450 1300 50  0001 C CNN
+F 0 "#PWR036" H 4450 1300 50  0001 C CNN
 F 1 "+3V3" H 4465 1623 50  0000 C CNN
 F 2 "" H 4450 1450 50  0001 C CNN
@@
 	4450 1450 4450 1500
 $Comp
-L AR2ISS:C C?
+L AR2ISS:C C10
 U 1 1 609F7991
 P 4700 1750
-F 0 "C?" H 4815 1796 50  0000 L CNN
+F 0 "C10" H 4815 1796 50  0000 L CNN
 F 1 "100n" H 4815 1705 50  0000 L CNN
-F 2 "" H 4738 1600 50  0001 C CNN
+F 2 "Capacitor_SMD:C_0603_1608Metric" H 4738 1600 50  0001 C CNN
 F 3 "~" H 4700 1750 50  0001 C CNN
 	1    4700 1750
@@
 $EndComp
 $Comp
-L power:GND #PWR?
+L power:GND #PWR038
 U 1 1 609F854C
 P 4700 2000
-F 0 "#PWR?" H 4700 1750 50  0001 C CNN
+F 0 "#PWR038" H 4700 1750 50  0001 C CNN
 F 1 "GND" H 4705 1827 50  0000 C CNN
 F 2 "" H 4700 2000 50  0001 C CNN
@@
 	5250 4050 6600 4050
 $Comp
-L Connector:DB9_Female J?
+L Connector:DB9_Female J8
 U 1 1 609FDDEA
 P 10150 3650
-F 0 "J?" H 10330 3696 50  0000 L CNN
+F 0 "J8" H 10330 3696 50  0000 L CNN
 F 1 "DB9_Female" H 10330 3605 50  0000 L CNN
 F 2 "" H 10150 3650 50  0001 C CNN
@@
 $EndComp
 $Comp
-L Connector_Generic:Conn_02x03_Odd_Even J?
+L Connector_Generic:Conn_02x03_Odd_Even J6
 U 1 1 60A00C31
 P 8800 3550
-F 0 "J?" V 8896 3362 50  0000 R CNN
+F 0 "J6" V 8896 3362 50  0000 R CNN
 F 1 "Conn_02x03_Odd_Even" V 8805 3362 50  0000 R CNN
 F 2 "" H 8800 3550 50  0001 C CNN
@@
 	7200 3650 8300 3650
 $Comp
-L power:GND #PWR?
+L power:GND #PWR041
 U 1 1 60A12D1E
 P 9750 4200
-F 0 "#PWR?" H 9750 3950 50  0001 C CNN
+F 0 "#PWR041" H 9750 3950 50  0001 C CNN
 F 1 "GND" H 9755 4027 50  0000 C CNN
 F 2 "" H 9750 4200 50  0001 C CNN
@@
 	9750 4050 9850 4050
 $Comp
-L Connector_Generic:Conn_01x03 J?
+L Connector_Generic:Conn_01x03 J7
 U 1 1 60A1513D
 P 10050 5050
-F 0 "J?" H 10130 5092 50  0000 L CNN
+F 0 "J7" H 10130 5092 50  0000 L CNN
 F 1 "Conn_01x03" H 10130 5001 50  0000 L CNN
 F 2 "" H 10050 5050 50  0001 C CNN
@@
 	7650 4050 7200 4050
 $Comp
-L power:GND #PWR?
+L power:GND #PWR042
 U 1 1 60A1743F
 P 9750 5300
-F 0 "#PWR?" H 9750 5050 50  0001 C CNN
+F 0 "#PWR042" H 9750 5050 50  0001 C CNN
 F 1 "GND" H 9755 5127 50  0000 C CNN
 F 2 "" H 9750 5300 50  0001 C CNN

Commit message: placement
Parts:
- J6: footprint (none) -> Connector_PinHeader_2.54mm:PinHeader_2x03_P2.54mm_Vertical
- J8: footprint (none) -> Mouser:23117651
Connections:
- net RS232Filter/A_ext renamed RS232Filter_1/A_int
- net RS232Filter/A_int renamed RS232Filter_1/A_ext
- net RS232Filter/B_ext renamed RS232Filter_1/B_int
- net RS232Filter/B_int renamed RS232Filter_1/B_ext
- net RS232Filter/Y_ext renamed sheet608DD623/A_int
- net RS232Filter/Y_int renamed sheet608DD623/A_ext
- net RS232Filter/Z_ext renamed sheet608DD623/B_int
- net RS232Filter/Z_int renamed sheet608DD623/B_ext
Changed lines of the file:
@@
 $Descr A4 11693 8268
 encoding utf-8
-Sheet 4 21
+Sheet 4 22
 Title ""
 Date ""
@@
 Wire Wire Line
 	2250 4050 3650 4050
-$Sheet
-S 6600 3350 600  800
-U 609FB88E
-F0 "RS232Filter" 50
-F1 "RS422Filter.sch" 50
-F2 "A_ext" I L 6600 3650 50
-F3 "B_ext" I L 6600 3450 50
-F4 "A_int" I R 7200 3650 50
-F5 "B_int" I R 7200 3450 50
-F6 "Y_ext" I L 6600 4050 50
-F7 "Z_ext" I L 6600 3850 50
-F8 "Y_int" I R 7200 4050 50
-F9 "Z_int" I R 7200 3850 50
-$EndSheet
 Wire Wire Line
 	6600 3450 5250 3450
 Wire Wire Line
 	5250 3650 6600 3650
-Wire Wire Line
-	6600 3850 5250 3850
-Wire Wire Line
-	5250 4050 6600 4050
 $Comp
 L Connector:DB9_Female J8
@@
 F 0 "J8" H 10330 3696 50  0000 L CNN
 F 1 "DB9_Female" H 10330 3605 50  0000 L CNN
-F 2 "" H 10150 3650 50  0001 C CNN
+F 2 "Mouser:23117651" H 10150 3650 50  0001 C CNN
 F 3 " ~" H 10150 3650 50  0001 C CNN
 	1    10150 3650
@@
 F 0 "J6" V 8896 3362 50  0000 R CNN
 F 1 "Conn_02x03_Odd_Even" V 8805 3362 50  0000 R CNN
-F 2 "" H 8800 3550 50  0001 C CNN
+F 2 "Connector_PinHeader_2.54mm:PinHeader_2x03_P2.54mm_Vertical" H 8800 3550 50  0001 C CNN
 F 3 "~" H 8800 3550 50  0001 C CNN
 	1    8800 3550
@@
 $EndComp
 Wire Wire Line
-	7200 3850 7800 3850
-Wire Wire Line
-	7650 4050 7200 4050
+	7650 4250 7200 4250
 $Comp
 L power:GND #PWR042
@@
 	9750 5150 9850 5150
 Wire Wire Line
-	7800 3850 7800 4950
+	7800 4050 7800 4950
 Wire Wire Line
 	7800 4950 9850 4950
 Wire Wire Line
 	7650 5050 9850 5050
-Wire Wire Line
-	7650 4050 7650 5050
+$Sheet
+S 6600 3350 600  400
+U 609FB88E
+F0 "RS232Filter_1" 50
+F1 "RS422Filter.sch" 50
+F2 "B_ext" I R 7200 3450 50
+F3 "A_int" I L 6600 3650 50
+F4 "B_int" I L 6600 3450 50
+F5 "A_ext" I R 7200 3650 50
+$EndSheet
+$Sheet
+S 6600 3950 600  400
+U 608DD62D
+F0 "sheet608DD623" 50
+F1 "RS422Filter.sch" 50
+F2 "B_ext" I R 7200 4050 50
+F3 "A_int" I L 6600 4250 50
+F4 "B_int" I L 6600 4050 50
+F5 "A_ext" I R 7200 4250 50
+$EndSheet
+Wire Wire Line
+	7650 4250 7650 5050
+Wire Wire Line
+	7200 4050 7800 4050
+Wire Wire Line
+	6600 4050 6150 4050
+Wire Wire Line
+	6150 4050 6150 3850
+Wire Wire Line
+	6150 3850 5250 3850
+Wire Wire Line
+	5250 4050 6000 4050
+Wire Wire Line
+	6000 4050 6000 4250
+Wire Wire Line
+	6000 4250 6600 4250
 $EndSCHEMATC

Commit message: add TLE5602
Parts:
- J8: footprint Mouser:23117651 -> AR2ISS:L177TSEH09SOL2RM8
Changed lines of the file:
@@
 $Descr A4 11693 8268
 encoding utf-8
-Sheet 4 22
+Sheet 3 22
 Title ""
 Date ""
@@
 F 0 "J8" H 10330 3696 50  0000 L CNN
 F 1 "DB9_Female" H 10330 3605 50  0000 L CNN
-F 2 "Mouser:23117651" H 10150 3650 50  0001 C CNN
+F 2 "AR2ISS:L177TSEH09SOL2RM8" H 10150 3650 50  0001 C CNN
 F 3 " ~" H 10150 3650 50  0001 C CNN
 	1    10150 3650

Commit message: placement, routing
Parts:
- J7: footprint (none) -> Connector_PinHeader_2.54mm:PinHeader_1x03_P2.54mm_Vertical
Changed lines of the file:
@@
 F 0 "J7" H 10130 5092 50  0000 L CNN
 F 1 "Conn_01x03" H 10130 5001 50  0000 L CNN
-F 2 "" H 10050 5050 50  0001 C CNN
+F 2 "Connector_PinHeader_2.54mm:PinHeader_1x03_P2.54mm_Vertical" H 10050 5050 50  0001 C CNN
 F 3 "~" H 10050 5050 50  0001 C CNN
 	1    10050 5050

Commit message: ready for jlc
Connections:
- net RS232Filter_1/A_int: now also U1.13 (R1IN); no longer U1.7 (T2OUT)
- net sheet608DD623/B_int: now also U1.7 (T2OUT); no longer U1.13 (R1IN)
Changed lines of the file:
@@
 Wire Wire Line
 	6600 3450 5250 3450
-Wire Wire Line
-	5250 3650 6600 3650
 $Comp
 L Connector:DB9_Female J8
@@
 	6600 4050 6150 4050
 Wire Wire Line
-	6150 4050 6150 3850
-Wire Wire Line
-	6150 3850 5250 3850
-Wire Wire Line
 	5250 4050 6000 4050
 Wire Wire Line
@@
 Wire Wire Line
 	6000 4250 6600 4250
+Wire Wire Line
+	5250 3650 6150 3650
+Wire Wire Line
+	6150 3650 6150 4050
+Wire Wire Line
+	5250 3850 6350 3850
+Wire Wire Line
+	6350 3850 6350 3650
+Wire Wire Line
+	6350 3650 6600 3650
 $EndSCHEMATC
