File: RS422.sch (KiCad schematic (older format))
At the start: 30 parts

Commit message: add SDcard, OneWire, Batt, analog out, digital out
Parts:
- R?: value 1k -> 3k
Connections:
- wire segments 188 -> 190
Other:
- moved on the sheet: R?
Changed lines of the file:
@@
 $Descr A4 11693 8268
 encoding utf-8
-Sheet 7 10
+Sheet 6 19
 Title ""
 Date ""
@@
 L AR2ISS:R R?
 U 1 1 60AB256C
-P 5800 5500
-F 0 "R?" H 5870 5546 50  0000 L CNN
-F 1 "1k" H 5870 5455 50  0000 L CNN
-F 2 "" V 5730 5500 50  0001 C CNN
-F 3 "~" H 5800 5500 50  0001 C CNN
-	1    5800 5500
+P 6350 4750
+F 0 "R?" H 6420 4796 50  0000 L CNN
+F 1 "3k" H 6420 4705 50  0000 L CNN
+F 2 "" V 6280 4750 50  0001 C CNN
+F 3 "~" H 6350 4750 50  0001 C CNN
+	1    6350 4750
 	1    0    0    -1
 $EndComp
@@
 Wire Wire Line
 	5800 5150 6100 5150
-Text Label 5800 5300 0    50   ~ 0
+Text Label 6350 4950 3    50   ~ 0
 DE3
 $Comp
@@
 	1    0    0    -1
 $EndComp
-Wire Wire Line
-	5800 5300 5800 5350
 Wire Wire Line
 	6550 5100 6550 5700
@@
 Connection ~ 5800 3900
 Wire Wire Line
-	5500 4500 6550 4500
+	5500 4500 6350 4500
 Wire Wire Line
 	5800 5700 6550 5700
@@
 Wire Wire Line
 	3750 7000 3000 7000
+Wire Wire Line
+	6350 4600 6350 4500
+Connection ~ 6350 4500
+Wire Wire Line
+	6350 4500 6550 4500
+Wire Wire Line
+	6350 4900 6350 4950
 $EndSCHEMATC

Commit message: start placement
Parts:
- removed C? (x4): 100n, symbol AR2ISS:C
- removed J?: RJ45_LED_Shielded, symbol Connector:RJ45_LED_Shielded
- removed R? (x8): 10k, symbol AR2ISS:R
- removed R? (x2): 3k, symbol AR2ISS:R
- removed R? (x6): 1k, symbol AR2ISS:R
- removed U? (x4): SN75176AD, Package_SO:SOIC-8_3.9x4.9mm_P1.27mm, symbol Interface_UART:SN75176AD
- added J15: RJ45_LED, AR2ISS:RJ45_LED, symbol AR2ISS:RJ45_LED
- C22: renamed from C?; footprint (none) -> Capacitor_SMD:C_0603_1608Metric
- L9: renamed from L?; footprint (none) -> Inductor_SMD:L_0603_1608Metric
- R43, R44, R45: renamed from R?; footprint (none) -> Resistor_SMD:R_0603_1608Metric
Connections:
- net labels added: PTT1, PTT2
- net labels removed: DE1, DE2, DE3, DE4, RX2, TX2
- wire segments 190 -> 71
Other:
- moved on the sheet: C22, R43, R44, R45

Commit message: add TLE5602
Changed lines of the file:
@@
 $Descr A4 11693 8268
 encoding utf-8
-Sheet 18 22
+Sheet 16 22
 Title ""
 Date ""
@@
 	6150 1500 6150 1400
 Connection ~ 6150 1400
-Text HLabel 5950 6850 2    50   Input ~ 0
-PTT2
 Text HLabel 5950 5150 2    50   Input ~ 0
-PTT1
-Text HLabel 5950 3350 2    50   Input ~ 0
+TX2
+Text HLabel 5950 3350 2    50   Output ~ 0
 RX
 Wire Wire Line
@@
 F2 "A_in" I L 5150 4900 50
 F3 "B_in" I L 5150 5300 50
-F4 "MODE" I R 5850 5300 50
+F4 "MODE" I R 5850 5000 50
 F5 "VCC" I R 5850 4900 50
 F6 "DATA" B R 5850 5150 50
@@
 	6200 3500 5850 3500
 $Comp
-L power:GND #PWR060
-U 1 1 607B0400
-P 6200 5550
-F 0 "#PWR060" H 6200 5300 50  0001 C CNN
-F 1 "GND" H 6205 5377 50  0000 C CNN
-F 2 "" H 6200 5550 50  0001 C CNN
-F 3 "" H 6200 5550 50  0001 C CNN
-	1    6200 5550
-	1    0    0    -1
-$EndComp
-Wire Wire Line
-	6200 5550 6200 5300
-Wire Wire Line
-	6200 5300 5850 5300
-$Comp
 L power:GND #PWR061
 U 1 1 607B1C3E
@@
 Wire Wire Line
 	2200 3800 2550 3800
+Text HLabel 5950 6850 2    50   Output ~ 0
+RX2
+Wire Wire Line
+	5850 5000 6150 5000
+Wire Wire Line
+	6150 5000 6150 4900
+Connection ~ 6150 4900
 $EndSCHEMATC

Commit message: routing
Connections:
- net at J15.13: now also C22.2, R45.2
Changed lines of the file:
@@
 F6 "DATA" B R 5850 3350 50
 $EndSheet
-Wire Wire Line
-	2200 3800 2550 3800
 Text HLabel 5950 6850 2    50   Output ~ 0
 RX2
@@
 	6150 5000 6150 4900
 Connection ~ 6150 4900
+Wire Wire Line
+	2400 3800 2550 3800
+Wire Wire Line
+	2400 3800 2200 3800
+Connection ~ 2400 3800
 $EndSCHEMATC

Commit message: routing
Connections:
- net RS485Tranceiver1/MODE renamed VCC_RS422
Changed lines of the file:
@@
 	2400 3800 2200 3800
 Connection ~ 2400 3800
+Text Label 6500 1200 0    50   ~ 0
+VCC_RS422
 $EndSCHEMATC
