File: RS485Tranceiver.sch (KiCad schematic (older format))
At the start: 19 parts, among them J10 Conn_01x02, U13 SN75176AD

Commit message: placement
Connections:
- net A_in: now also D9.2 (A2), J10.2 (Pin_2), L13.2; no longer L11.1
- net B_in: now also D9.1 (A1), L12.2, R66.1; no longer L10.1
- net at R68.2, R69.1, U13.6 (A): now also L11.1; no longer D9.2 (A2), J10.2 (Pin_2), L13.2
- net at R67.2, R68.1, U13.7 (B): now also L10.1; no longer D9.1 (A1), L12.2, R66.1
Other:
- moved on the sheet: C28, C29, C30, C31, D27, J12, L14, L15, L16, L17, R53, R54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

Commit message: add TLE5602
Changed lines of the file:
@@
 $Descr A4 11693 8268
 encoding utf-8
-Sheet 20 22
+Sheet 21 22
 Title ""
 Date ""
@@
 AR Path="/608DA584/60797D2F/6072BD51" Ref="U5"  Part="1"
 AR Path="/608DA584/607938CE/6072BD51" Ref="U19"  Part="1"
-F 0 "U4" H 8600 2981 50  0000 C CNN
+F 0 "U19" H 8600 2981 50  0000 C CNN
 F 1 "SN75176AD" H 8600 2890 50  0000 C CNN
 F 2 "Package_SO:SOIC-8_3.9x4.9mm_P1.27mm" H 8600 1900 50  0001 C CNN
@@
 AR Path="/608DA584/60797D2F/6072BD57" Ref="R65"  Part="1"
 AR Path="/608DA584/607938CE/6072BD57" Ref="R72"  Part="1"
-F 0 "R58" H 8020 2996 50  0000 L CNN
+F 0 "R72" H 8020 2996 50  0000 L CNN
 F 1 "10k" H 8020 2905 50  0000 L CNN
 F 2 "Resistor_SMD:R_0603_1608Metric" V 7880 2950 50  0001 C CNN
@@
 AR Path="/608DA584/60797D2F/6072BD5D" Ref="R66"  Part="1"
 AR Path="/608DA584/607938CE/6072BD5D" Ref="R103"  Part="1"
-F 0 "R59" H 10370 2996 50  0000 L CNN
+F 0 "R103" H 10370 2996 50  0000 L CNN
 F 1 "3k" H 10370 2905 50  0000 L CNN
 F 2 "Resistor_SMD:R_0603_1608Metric" V 10230 2950 50  0001 C CNN
@@
 AR Path="/608DA584/60797D2F/6072BD63" Ref="R63"  Part="1"
 AR Path="/608DA584/607938CE/6072BD63" Ref="R70"  Part="1"
-F 0 "R56" H 8020 2196 50  0000 L CNN
+F 0 "R70" H 8020 2196 50  0000 L CNN
 F 1 "10k" H 8020 2105 50  0000 L CNN
 F 2 "Resistor_SMD:R_0603_1608Metric" V 7880 2150 50  0001 C CNN
@@
 AR Path="/608DA584/60797D2F/6072BD8E" Ref="C37"  Part="1"
 AR Path="/608DA584/607938CE/6072BD8E" Ref="C42"  Part="1"
-F 0 "C32" H 9765 2446 50  0000 L CNN
+F 0 "C42" H 9765 2446 50  0000 L CNN
 F 1 "100n" H 9765 2355 50  0000 L CNN
 F 2 "Capacitor_SMD:C_0603_1608Metric" H 9688 2250 50  0001 C CNN
@@
 AR Path="/608DA584/60797D2F/6072BDA0" Ref="R64"  Part="1"
 AR Path="/608DA584/607938CE/6072BDA0" Ref="R71"  Part="1"
-F 0 "R57" H 8020 2596 50  0000 L CNN
+F 0 "R71" H 8020 2596 50  0000 L CNN
 F 1 "1k" H 8020 2505 50  0000 L CNN
 F 2 "Resistor_SMD:R_0603_1608Metric" V 7880 2550 50  0001 C CNN
@@
 AR Path="/608DA584/60797D2F/6073EDBE" Ref="D28"  Part="1"
 AR Path="/608DA584/607938CE/6073EDBE" Ref="D29"  Part="1"
-F 0 "D27" V 2354 2630 50  0000 L CNN
+F 0 "D29" V 2354 2630 50  0000 L CNN
 F 1 "PESD2CAN" V 2445 2630 50  0000 L CNN
 F 2 "Package_TO_SOT_SMD:SOT-23_Handsoldering" H 2250 2550 50  0001 C CNN
@@
 AR Path="/608DA584/60797D2F/6073EDC4" Ref="L20"  Part="1"
 AR Path="/608DA584/607938CE/6073EDC4" Ref="L24"  Part="1"
-F 0 "L16" V 4740 1800 50  0000 C CNN
+F 0 "L24" V 4740 1800 50  0000 C CNN
 F 1 "74279266" V 4649 1800 50  0000 C CNN
 F 2 "Inductor_SMD:L_0603_1608Metric" H 4550 1800 50  0001 C CNN
@@
 AR Path="/608DA584/60797D2F/6073EDCA" Ref="R60"  Part="1"
 AR Path="/608DA584/607938CE/6073EDCA" Ref="R67"  Part="1"
-F 0 "R53" H 5470 2146 50  0000 L CNN
+F 0 "R67" H 5470 2146 50  0000 L CNN
 F 1 "221" H 5470 2055 50  0000 L CNN
 F 2 "Resistor_SMD:R_0603_1608Metric" V 5330 2100 50  0001 C CNN
@@
 AR Path="/608DA584/60797D2F/6073EDD0" Ref="C35"  Part="1"
 AR Path="/608DA584/607938CE/6073EDD0" Ref="C40"  Part="1"
-F 0 "C30" H 5515 2546 50  0000 L CNN
+F 0 "C40" H 5515 2546 50  0000 L CNN
 F 1 "1n" H 5515 2455 50  0000 L CNN
 F 2 "Capacitor_SMD:C_0603_1608Metric" H 5438 2350 50  0001 C CNN
@@
 AR Path="/608DA584/60797D2F/6073EDD6" Ref="C33"  Part="1"
 AR Path="/608DA584/607938CE/6073EDD6" Ref="C38"  Part="1"
-F 0 "C28" H 6015 2146 50  0000 L CNN
+F 0 "C38" H 6015 2146 50  0000 L CNN
 F 1 "470p" H 6015 2055 50  0000 L CNN
 F 2 "Capacitor_SMD:C_0603_1608Metric" H 5938 1950 50  0001 C CNN
@@
 AR Path="/608DA584/60797D2F/6073EDDC" Ref="L18"  Part="1"
 AR Path="/608DA584/607938CE/6073EDDC" Ref="L22"  Part="1"
-F 0 "L14" V 6940 1800 50  0000 C CNN
+F 0 "L22" V 6940 1800 50  0000 C CNN
 F 1 "10u" V 6849 1800 50  0000 C CNN
 F 2 "Inductor_SMD:L_0603_1608Metric" H 6750 1800 50  0001 C CNN
@@
 AR Path="/608DA584/60797D2F/6073EDF8" Ref="L21"  Part="1"
 AR Path="/608DA584/607938CE/6073EDF8" Ref="L25"  Part="1"
-F 0 "L17" V 4740 3300 50  0000 C CNN
+F 0 "L25" V 4740 3300 50  0000 C CNN
 F 1 "74279266" V 4649 3300 50  0000 C CNN
 F 2 "Inductor_SMD:L_0603_1608Metric" H 4550 3300 50  0001 C CNN
@@
 AR Path="/608DA584/60797D2F/6073EDFE" Ref="R61"  Part="1"
 AR Path="/608DA584/607938CE/6073EDFE" Ref="R68"  Part="1"
-F 0 "R54" H 5470 3646 50  0000 L CNN
+F 0 "R68" H 5470 3646 50  0000 L CNN
 F 1 "221" H 5470 3555 50  0000 L CNN
 F 2 "Resistor_SMD:R_0603_1608Metric" V 5330 3600 50  0001 C CNN
@@
 AR Path="/608DA584/60797D2F/6073EE04" Ref="C36"  Part="1"
 AR Path="/608DA584/607938CE/6073EE04" Ref="C41"  Part="1"
-F 0 "C31" H 5515 4046 50  0000 L CNN
+F 0 "C41" H 5515 4046 50  0000 L CNN
 F 1 "1n" H 5515 3955 50  0000 L CNN
 F 2 "Capacitor_SMD:C_0603_1608Metric" H 5438 3850 50  0001 C CNN
@@
 AR Path="/608DA584/60797D2F/6073EE0A" Ref="C34"  Part="1"
 AR Path="/608DA584/607938CE/6073EE0A" Ref="C39"  Part="1"
-F 0 "C29" H 6015 3646 50  0000 L CNN
+F 0 "C39" H 6015 3646 50  0000 L CNN
 F 1 "470p" H 6015 3555 50  0000 L CNN
 F 2 "Capacitor_SMD:C_0603_1608Metric" H 5938 3450 50  0001 C CNN
@@
 AR Path="/608DA584/60797D2F/6073EE10" Ref="L19"  Part="1"
 AR Path="/608DA584/607938CE/6073EE10" Ref="L23"  Part="1"
-F 0 "L15" V 6940 3300 50  0000 C CNN
+F 0 "L23" V 6940 3300 50  0000 C CNN
 F 1 "10u" V 6849 3300 50  0000 C CNN
 F 2 "Inductor_SMD:L_0603_1608Metric" H 6750 3300 50  0001 C CNN
@@
 AR Path="/608DA584/60797D2F/6073EE40" Ref="R62"  Part="1"
 AR Path="/608DA584/607938CE/6073EE40" Ref="R69"  Part="1"
-F 0 "R55" H 3470 2196 50  0000 L CNN
+F 0 "R69" H 3470 2196 50  0000 L CNN
 F 1 "120" H 3470 2105 50  0000 L CNN
 F 2 "Resistor_SMD:R_0603_1608Metric" V 3330 2150 50  0001 C CNN
@@
 AR Path="/608DA584/60797D2F/6073EE46" Ref="J13"  Part="1"
 AR Path="/608DA584/607938CE/6073EE46" Ref="J14"  Part="1"
-F 0 "J12" H 3518 2867 50  0000 C CNN
+F 0 "J14" H 3518 2867 50  0000 C CNN
 F 1 "Conn_01x02" H 3518 2776 50  0000 C CNN
 F 2 "Connector_PinHeader_2.54mm:PinHeader_1x02_P2.54mm_Vertical" H 3600 2650 50  0001 C CNN

Commit message: routing
Parts:
- removed U13: SN75176AD, Package_SO:SOIC-8_3.9x4.9mm_P1.27mm, symbol Interface_UART:SN75176AD
- added U19: SP3485EN-L/TR, Package_SO:SOIC-8_3.9x4.9mm_P1.27mm, symbol Interface_UART:SP3485EN
- R67, R69: value 10k -> NB
- R68: value 1k -> NB
- R70: value 3k -> 4.7k
Connections:
- net DATA: now also U19.1 (RO), U19.4 (DI)
- net DE1: now also U19.2 (~RE~), U19.3 (DE)
- net GND: now also U19.5 (GND)
- net VCC: now also U19.8 (VCC)
- net at R68.2, R69.1: now also L10.1, U19.7 (B); no longer L11.1
- net at R67.2, R68.1: now also L11.1, U19.6 (A); no longer L10.1
Other:
- moved on the sheet: C23, C24, C25, C26, C27, J11, L10, L11, L12, L13, R46, R47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

Commit message: placement, routing
Changed lines of the file:
@@
 $Descr A4 11693 8268
 encoding utf-8
-Sheet 17 22
+Sheet 20 22
 Title ""
 Date ""
@@
 AR Path="/608DA584/60797D2F/6072BD57" Ref="R65"  Part="1"
 AR Path="/608DA584/607938CE/6072BD57" Ref="R72"  Part="1"
-F 0 "R51" H 8020 2996 50  0000 L CNN
+F 0 "R72" H 8020 2996 50  0000 L CNN
 F 1 "NB" H 8020 2905 50  0000 L CNN
 F 2 "Resistor_SMD:R_0603_1608Metric" V 7880 2950 50  0001 C CNN
@@
 AR Path="/608DA584/60797D2F/6072BD5D" Ref="R66"  Part="1"
 AR Path="/608DA584/607938CE/6072BD5D" Ref="R103"  Part="1"
-F 0 "R52" H 10370 2996 50  0000 L CNN
+F 0 "R103" H 10370 2996 50  0000 L CNN
 F 1 "4.7k" H 10370 2905 50  0000 L CNN
 F 2 "Resistor_SMD:R_0603_1608Metric" V 10230 2950 50  0001 C CNN
@@
 AR Path="/608DA584/60797D2F/6072BD63" Ref="R63"  Part="1"
 AR Path="/608DA584/607938CE/6072BD63" Ref="R70"  Part="1"
-F 0 "R49" H 8020 2196 50  0000 L CNN
+F 0 "R70" H 8020 2196 50  0000 L CNN
 F 1 "NB" H 8020 2105 50  0000 L CNN
 F 2 "Resistor_SMD:R_0603_1608Metric" V 7880 2150 50  0001 C CNN
@@
 AR Path="/608DA584/60797D2F/6072BD8E" Ref="C37"  Part="1"
 AR Path="/608DA584/607938CE/6072BD8E" Ref="C42"  Part="1"
-F 0 "C27" H 9765 2596 50  0000 L CNN
+F 0 "C42" H 9765 2596 50  0000 L CNN
 F 1 "100n" H 9765 2505 50  0000 L CNN
 F 2 "Capacitor_SMD:C_0603_1608Metric" H 9688 2400 50  0001 C CNN
@@
 AR Path="/608DA584/60797D2F/6072BDA0" Ref="R64"  Part="1"
 AR Path="/608DA584/607938CE/6072BDA0" Ref="R71"  Part="1"
-F 0 "R50" H 8020 2596 50  0000 L CNN
+F 0 "R71" H 8020 2596 50  0000 L CNN
 F 1 "NB" H 8020 2505 50  0000 L CNN
 F 2 "Resistor_SMD:R_0603_1608Metric" V 7880 2550 50  0001 C CNN
@@
 AR Path="/608DA584/60797D2F/6073EDBE" Ref="D28"  Part="1"
 AR Path="/608DA584/607938CE/6073EDBE" Ref="D29"  Part="1"
-F 0 "D24" V 2354 2630 50  0000 L CNN
+F 0 "D29" V 2354 2630 50  0000 L CNN
 F 1 "PESD2CAN" V 2445 2630 50  0000 L CNN
 F 2 "Package_TO_SOT_SMD:SOT-23_Handsoldering" H 2250 2550 50  0001 C CNN
@@
 AR Path="/608DA584/60797D2F/6073EDC4" Ref="L20"  Part="1"
 AR Path="/608DA584/607938CE/6073EDC4" Ref="L24"  Part="1"
-F 0 "L12" V 4740 3300 50  0000 C CNN
+F 0 "L24" V 4740 3300 50  0000 C CNN
 F 1 "74279266" V 4649 3300 50  0000 C CNN
 F 2 "Inductor_SMD:L_0603_1608Metric" H 4550 3300 50  0001 C CNN
@@
 AR Path="/608DA584/60797D2F/6073EDCA" Ref="R60"  Part="1"
 AR Path="/608DA584/607938CE/6073EDCA" Ref="R67"  Part="1"
-F 0 "R46" H 5470 3646 50  0000 L CNN
+F 0 "R67" H 5470 3646 50  0000 L CNN
 F 1 "221" H 5470 3555 50  0000 L CNN
 F 2 "Resistor_SMD:R_0603_1608Metric" V 5330 3600 50  0001 C CNN
@@
 AR Path="/608DA584/60797D2F/6073EDD0" Ref="C35"  Part="1"
 AR Path="/608DA584/607938CE/6073EDD0" Ref="C40"  Part="1"
-F 0 "C25" H 5515 4046 50  0000 L CNN
+F 0 "C40" H 5515 4046 50  0000 L CNN
 F 1 "1n" H 5515 3955 50  0000 L CNN
 F 2 "Capacitor_SMD:C_0603_1608Metric" H 5438 3850 50  0001 C CNN
@@
 AR Path="/608DA584/60797D2F/6073EDD6" Ref="C33"  Part="1"
 AR Path="/608DA584/607938CE/6073EDD6" Ref="C38"  Part="1"
-F 0 "C23" H 6015 3646 50  0000 L CNN
+F 0 "C38" H 6015 3646 50  0000 L CNN
 F 1 "470p" H 6015 3555 50  0000 L CNN
 F 2 "Capacitor_SMD:C_0603_1608Metric" H 5938 3450 50  0001 C CNN
@@
 AR Path="/608DA584/60797D2F/6073EDDC" Ref="L18"  Part="1"
 AR Path="/608DA584/607938CE/6073EDDC" Ref="L22"  Part="1"
-F 0 "L10" V 6940 3300 50  0000 C CNN
+F 0 "L22" V 6940 3300 50  0000 C CNN
 F 1 "10u" V 6849 3300 50  0000 C CNN
 F 2 "Inductor_SMD:L_0603_1608Metric" H 6750 3300 50  0001 C CNN
@@
 AR Path="/608DA584/60797D2F/6073EDF8" Ref="L21"  Part="1"
 AR Path="/608DA584/607938CE/6073EDF8" Ref="L25"  Part="1"
-F 0 "L13" V 4740 1800 50  0000 C CNN
+F 0 "L25" V 4740 1800 50  0000 C CNN
 F 1 "74279266" V 4649 1800 50  0000 C CNN
 F 2 "Inductor_SMD:L_0603_1608Metric" H 4550 1800 50  0001 C CNN
@@
 AR Path="/608DA584/60797D2F/6073EDFE" Ref="R61"  Part="1"
 AR Path="/608DA584/607938CE/6073EDFE" Ref="R68"  Part="1"
-F 0 "R47" H 5470 2146 50  0000 L CNN
+F 0 "R68" H 5470 2146 50  0000 L CNN
 F 1 "221" H 5470 2055 50  0000 L CNN
 F 2 "Resistor_SMD:R_0603_1608Metric" V 5330 2100 50  0001 C CNN
@@
 AR Path="/608DA584/60797D2F/6073EE04" Ref="C36"  Part="1"
 AR Path="/608DA584/607938CE/6073EE04" Ref="C41"  Part="1"
-F 0 "C26" H 5515 2546 50  0000 L CNN
+F 0 "C41" H 5515 2546 50  0000 L CNN
 F 1 "1n" H 5515 2455 50  0000 L CNN
 F 2 "Capacitor_SMD:C_0603_1608Metric" H 5438 2350 50  0001 C CNN
@@
 AR Path="/608DA584/60797D2F/6073EE0A" Ref="C34"  Part="1"
 AR Path="/608DA584/607938CE/6073EE0A" Ref="C39"  Part="1"
-F 0 "C24" H 6015 2146 50  0000 L CNN
+F 0 "C39" H 6015 2146 50  0000 L CNN
 F 1 "470p" H 6015 2055 50  0000 L CNN
 F 2 "Capacitor_SMD:C_0603_1608Metric" H 5938 1950 50  0001 C CNN
@@
 AR Path="/608DA584/60797D2F/6073EE10" Ref="L19"  Part="1"
 AR Path="/608DA584/607938CE/6073EE10" Ref="L23"  Part="1"
-F 0 "L11" V 6940 1800 50  0000 C CNN
+F 0 "L23" V 6940 1800 50  0000 C CNN
 F 1 "10u" V 6849 1800 50  0000 C CNN
 F 2 "Inductor_SMD:L_0603_1608Metric" H 6750 1800 50  0001 C CNN
@@
 AR Path="/608DA584/60797D2F/6073EE40" Ref="R62"  Part="1"
 AR Path="/608DA584/607938CE/6073EE40" Ref="R69"  Part="1"
-F 0 "R48" H 3470 2996 50  0000 L CNN
+F 0 "R69" H 3470 2996 50  0000 L CNN
 F 1 "120" H 3470 2905 50  0000 L CNN
 F 2 "Resistor_SMD:R_0603_1608Metric" V 3330 2950 50  0001 C CNN
@@
 AR Path="/608DA584/60797D2F/6073EE46" Ref="J13"  Part="1"
 AR Path="/608DA584/607938CE/6073EE46" Ref="J14"  Part="1"
-F 0 "J11" H 3518 2667 50  0000 C CNN
+F 0 "J14" H 3518 2667 50  0000 C CNN
 F 1 "Conn_01x02" H 3518 2576 50  0000 C CNN
 F 2 "Connector_PinHeader_2.54mm:PinHeader_1x02_P2.54mm_Vertical" H 3600 2450 50  0001 C CNN
@@
 AR Path="/608DA584/60795F15/60C746E7" Ref="U4"  Part="1"
 AR Path="/608DA584/60797D2F/60C746E7" Ref="U5"  Part="1"
-F 0 "U3" H 8700 3131 50  0000 C CNN
+F 0 "U19" H 8700 3131 50  0000 C CNN
 F 1 "SP3485EN-L/TR" H 8700 3040 50  0000 C CNN
 F 2 "Package_SO:SOIC-8_3.9x4.9mm_P1.27mm" H 9750 2200 50  0001 C CIN

Commit message: ready for jlc
Changed lines of the file:
@@
 $Descr A4 11693 8268
 encoding utf-8
-Sheet 20 22
+Sheet 16 22
 Title ""
 Date ""
@@
 AR Path="/608DA584/60797D2F/6072BD57" Ref="R65"  Part="1"
 AR Path="/608DA584/607938CE/6072BD57" Ref="R72"  Part="1"
-F 0 "R72" H 8020 2996 50  0000 L CNN
+F 0 "R51" H 8020 2996 50  0000 L CNN
 F 1 "NB" H 8020 2905 50  0000 L CNN
 F 2 "Resistor_SMD:R_0603_1608Metric" V 7880 2950 50  0001 C CNN
@@
 AR Path="/608DA584/60797D2F/6072BD5D" Ref="R66"  Part="1"
 AR Path="/608DA584/607938CE/6072BD5D" Ref="R103"  Part="1"
-F 0 "R103" H 10370 2996 50  0000 L CNN
+F 0 "R52" H 10370 2996 50  0000 L CNN
 F 1 "4.7k" H 10370 2905 50  0000 L CNN
 F 2 "Resistor_SMD:R_0603_1608Metric" V 10230 2950 50  0001 C CNN
@@
 AR Path="/608DA584/60797D2F/6072BD63" Ref="R63"  Part="1"
 AR Path="/608DA584/607938CE/6072BD63" Ref="R70"  Part="1"
-F 0 "R70" H 8020 2196 50  0000 L CNN
+F 0 "R49" H 8020 2196 50  0000 L CNN
 F 1 "NB" H 8020 2105 50  0000 L CNN
 F 2 "Resistor_SMD:R_0603_1608Metric" V 7880 2150 50  0001 C CNN
@@
 AR Path="/608DA584/60797D2F/6072BD8E" Ref="C37"  Part="1"
 AR Path="/608DA584/607938CE/6072BD8E" Ref="C42"  Part="1"
-F 0 "C42" H 9765 2596 50  0000 L CNN
+F 0 "C27" H 9765 2596 50  0000 L CNN
 F 1 "100n" H 9765 2505 50  0000 L CNN
 F 2 "Capacitor_SMD:C_0603_1608Metric" H 9688 2400 50  0001 C CNN
@@
 AR Path="/608DA584/60797D2F/6072BDA0" Ref="R64"  Part="1"
 AR Path="/608DA584/607938CE/6072BDA0" Ref="R71"  Part="1"
-F 0 "R71" H 8020 2596 50  0000 L CNN
+F 0 "R50" H 8020 2596 50  0000 L CNN
 F 1 "NB" H 8020 2505 50  0000 L CNN
 F 2 "Resistor_SMD:R_0603_1608Metric" V 7880 2550 50  0001 C CNN
@@
 AR Path="/608DA584/60797D2F/6073EDBE" Ref="D28"  Part="1"
 AR Path="/608DA584/607938CE/6073EDBE" Ref="D29"  Part="1"
-F 0 "D29" V 2354 2630 50  0000 L CNN
+F 0 "D24" V 2354 2630 50  0000 L CNN
 F 1 "PESD2CAN" V 2445 2630 50  0000 L CNN
 F 2 "Package_TO_SOT_SMD:SOT-23_Handsoldering" H 2250 2550 50  0001 C CNN
@@
 AR Path="/608DA584/60797D2F/6073EDC4" Ref="L20"  Part="1"
 AR Path="/608DA584/607938CE/6073EDC4" Ref="L24"  Part="1"
-F 0 "L24" V 4740 3300 50  0000 C CNN
+F 0 "L12" V 4740 3300 50  0000 C CNN
 F 1 "74279266" V 4649 3300 50  0000 C CNN
 F 2 "Inductor_SMD:L_0603_1608Metric" H 4550 3300 50  0001 C CNN
@@
 AR Path="/608DA584/60797D2F/6073EDCA" Ref="R60"  Part="1"
 AR Path="/608DA584/607938CE/6073EDCA" Ref="R67"  Part="1"
-F 0 "R67" H 5470 3646 50  0000 L CNN
+F 0 "R46" H 5470 3646 50  0000 L CNN
 F 1 "221" H 5470 3555 50  0000 L CNN
 F 2 "Resistor_SMD:R_0603_1608Metric" V 5330 3600 50  0001 C CNN
@@
 AR Path="/608DA584/60797D2F/6073EDD0" Ref="C35"  Part="1"
 AR Path="/608DA584/607938CE/6073EDD0" Ref="C40"  Part="1"
-F 0 "C40" H 5515 4046 50  0000 L CNN
+F 0 "C25" H 5515 4046 50  0000 L CNN
 F 1 "1n" H 5515 3955 50  0000 L CNN
 F 2 "Capacitor_SMD:C_0603_1608Metric" H 5438 3850 50  0001 C CNN
@@
 AR Path="/608DA584/60797D2F/6073EDD6" Ref="C33"  Part="1"
 AR Path="/608DA584/607938CE/6073EDD6" Ref="C38"  Part="1"
-F 0 "C38" H 6015 3646 50  0000 L CNN
+F 0 "C23" H 6015 3646 50  0000 L CNN
 F 1 "470p" H 6015 3555 50  0000 L CNN
 F 2 "Capacitor_SMD:C_0603_1608Metric" H 5938 3450 50  0001 C CNN
@@
 AR Path="/608DA584/60797D2F/6073EDDC" Ref="L18"  Part="1"
 AR Path="/608DA584/607938CE/6073EDDC" Ref="L22"  Part="1"
-F 0 "L22" V 6940 3300 50  0000 C CNN
+F 0 "L10" V 6940 3300 50  0000 C CNN
 F 1 "10u" V 6849 3300 50  0000 C CNN
 F 2 "Inductor_SMD:L_0603_1608Metric" H 6750 3300 50  0001 C CNN
@@
 AR Path="/608DA584/60797D2F/6073EDF8" Ref="L21"  Part="1"
 AR Path="/608DA584/607938CE/6073EDF8" Ref="L25"  Part="1"
-F 0 "L25" V 4740 1800 50  0000 C CNN
+F 0 "L13" V 4740 1800 50  0000 C CNN
 F 1 "74279266" V 4649 1800 50  0000 C CNN
 F 2 "Inductor_SMD:L_0603_1608Metric" H 4550 1800 50  0001 C CNN
@@
 AR Path="/608DA584/60797D2F/6073EDFE" Ref="R61"  Part="1"
 AR Path="/608DA584/607938CE/6073EDFE" Ref="R68"  Part="1"
-F 0 "R68" H 5470 2146 50  0000 L CNN
+F 0 "R47" H 5470 2146 50  0000 L CNN
 F 1 "221" H 5470 2055 50  0000 L CNN
 F 2 "Resistor_SMD:R_0603_1608Metric" V 5330 2100 50  0001 C CNN
@@
 AR Path="/608DA584/60797D2F/6073EE04" Ref="C36"  Part="1"
 AR Path="/608DA584/607938CE/6073EE04" Ref="C41"  Part="1"
-F 0 "C41" H 5515 2546 50  0000 L CNN
+F 0 "C26" H 5515 2546 50  0000 L CNN
 F 1 "1n" H 5515 2455 50  0000 L CNN
 F 2 "Capacitor_SMD:C_0603_1608Metric" H 5438 2350 50  0001 C CNN
@@
 AR Path="/608DA584/60797D2F/6073EE0A" Ref="C34"  Part="1"
 AR Path="/608DA584/607938CE/6073EE0A" Ref="C39"  Part="1"
-F 0 "C39" H 6015 2146 50  0000 L CNN
+F 0 "C24" H 6015 2146 50  0000 L CNN
 F 1 "470p" H 6015 2055 50  0000 L CNN
 F 2 "Capacitor_SMD:C_0603_1608Metric" H 5938 1950 50  0001 C CNN
@@
 AR Path="/608DA584/60797D2F/6073EE10" Ref="L19"  Part="1"
 AR Path="/608DA584/607938CE/6073EE10" Ref="L23"  Part="1"
-F 0 "L23" V 6940 1800 50  0000 C CNN
+F 0 "L11" V 6940 1800 50  0000 C CNN
 F 1 "10u" V 6849 1800 50  0000 C CNN
 F 2 "Inductor_SMD:L_0603_1608Metric" H 6750 1800 50  0001 C CNN
@@
 AR Path="/608DA584/60797D2F/6073EE40" Ref="R62"  Part="1"
 AR Path="/608DA584/607938CE/6073EE40" Ref="R69"  Part="1"
-F 0 "R69" H 3470 2996 50  0000 L CNN
+F 0 "R48" H 3470 2996 50  0000 L CNN
 F 1 "120" H 3470 2905 50  0000 L CNN
 F 2 "Resistor_SMD:R_0603_1608Metric" V 3330 2950 50  0001 C CNN
@@
 AR Path="/608DA584/60797D2F/6073EE46" Ref="J13"  Part="1"
 AR Path="/608DA584/607938CE/6073EE46" Ref="J14"  Part="1"
-F 0 "J14" H 3518 2667 50  0000 C CNN
+F 0 "J11" H 3518 2667 50  0000 C CNN
 F 1 "Conn_01x02" H 3518 2576 50  0000 C CNN
 F 2 "Connector_PinHeader_2.54mm:PinHeader_1x02_P2.54mm_Vertical" H 3600 2450 50  0001 C CNN
@@
 AR Path="/608DA584/60795F15/60C746E7" Ref="U4"  Part="1"
 AR Path="/608DA584/60797D2F/60C746E7" Ref="U5"  Part="1"
-F 0 "U19" H 8700 3131 50  0000 C CNN
+F 0 "U3" H 8700 3131 50  0000 C CNN
 F 1 "SP3485EN-L/TR" H 8700 3040 50  0000 C CNN
 F 2 "Package_SO:SOIC-8_3.9x4.9mm_P1.27mm" H 9750 2200 50  0001 C CIN
