File: controller.sch (KiCad schematic (older format))
At the start: 9 parts

Commit message: start placement
Parts:
- added D22: MMSZ3V6CW, Diode_SMD:D_SOD-123, symbol Device:D_Zener
- added U2: NUCLEO144-H745ZI, Module:ST_Morpho_Connector_144_STLink, symbol AR2ISS:NUCLEO144-H745ZI
- BT1: renamed from BT?; footprint (none) -> Diode_SMD:D_SOD-123
- C68, C69: renamed from C?; footprint (none) -> Capacitor_SMD:C_0603_1608Metric
- R125, R126, R127: renamed from R?; footprint (none) -> Resistor_SMD:R_0603_1608Metric
- gave numbers to parts that had none: 3
Connections:
- net labels added: SD_#CS, SD_MISO, SD_MOSI, SD_SCK
- wire segments 32 -> 63
Other:
- moved on the sheet: J26, R127

Commit message: placement
Parts:
- J25: footprint (none) -> Connector_IDC:IDC-Header_2x03_P2.54mm_Vertical
- J26: footprint (none) -> Connector_PinHeader_2.54mm:PinHeader_1x02_P2.54mm_Vertical
Changed lines of the file:
@@
 $Descr A3 16535 11693
 encoding utf-8
-Sheet 14 21
+Sheet 15 22
 Title ""
 Date "2021-04-18"
@@
 F 0 "J25" H 3950 5567 50  0000 C CNN
 F 1 "Conn_02x03_Odd_Even" H 3950 5476 50  0000 C CNN
-F 2 "" H 3900 5250 50  0001 C CNN
+F 2 "Connector_IDC:IDC-Header_2x03_P2.54mm_Vertical" H 3900 5250 50  0001 C CNN
 F 3 "~" H 3900 5250 50  0001 C CNN
 	1    3900 5250
@@
 F 0 "J26" H 13080 7042 50  0000 L CNN
 F 1 "Conn_01x02" H 13080 6951 50  0000 L CNN
-F 2 "" H 13000 7050 50  0001 C CNN
+F 2 "Connector_PinHeader_2.54mm:PinHeader_1x02_P2.54mm_Vertical" H 13000 7050 50  0001 C CNN
 F 3 "~" H 13000 7050 50  0001 C CNN
 	1    13000 7050
@@
 Wire Wire Line
 	7900 1350 7900 1800
-Wire Bus Line
-	3550 2450 3550 3200
 Text HLabel 3500 8000 0    50   Input ~ 0
 SD_#CS
@@
 Text HLabel 3200 8550 0    50   Input ~ 0
 SD_SCK
+Wire Bus Line
+	3550 2450 3550 3200
 $EndSCHEMATC

Commit message: add TLE5602
Parts:
- added JP1, JP2: Jumper_NO_Small, symbol Device:Jumper_NO_Small
- added R144: 100, symbol AR2ISS:R
- D26: footprint (none) -> Diode_SMD:D_SOD-123
Connections:
- net labels added: ADC12V, ADC3V3, ADC5V, ADCPWR, COM_RX1, COM_RX2, COM_TX1, COM_TX2, DA_IN_LL0, DA_IN_LL1, DA_IN_LL2, DA_IN_LL3, DA_IN_LL4, DA_IN_LL5, DA_IN_LL6, DA_IN_LL7, DA_IN_LL[0..7], NRST, SCL_ext, SDA_ext, SDMMC_CD, SDMMC_CK, SDMMC_CMD, SDMMC_D0
- net labels removed: DA_IN_LL, SD_#CS, SD_MISO, SD_MOSI, SD_SCK
- wire segments 63 -> 143
Other:
- moved on the sheet: D22, U2

Commit message: routing
Parts:
- BT1: footprint Diode_SMD:D_SOD-123 -> (none)
- D26: value D_Schottky -> BAT54W-HG3-08
- R127: value 4k7 -> 4.7k
- R144: value 100 -> 100R
Changed lines of the file:
@@
 P 1500 5750
 F 0 "D26" V 1546 5670 50  0000 R CNN
-F 1 "D_Schottky" V 1455 5670 50  0000 R CNN
+F 1 "BAT54W-HG3-08" V 1455 5670 50  0000 R CNN
 F 2 "Diode_SMD:D_SOD-123" H 1500 5750 50  0001 C CNN
 F 3 "~" H 1500 5750 50  0001 C CNN
@@
 F 0 "BT1" H 1618 6746 50  0000 L CNN
 F 1 "Battery_Cell" H 1618 6655 50  0000 L CNN
-F 2 "Diode_SMD:D_SOD-123" V 1500 6710 50  0001 C CNN
+F 2 "" V 1500 6710 50  0001 C CNN
 F 3 "~" V 1500 6710 50  0001 C CNN
 	1    1500 6650
@@
 P 12450 6750
 F 0 "R127" H 12520 6796 50  0000 L CNN
-F 1 "4k7" H 12520 6705 50  0000 L CNN
+F 1 "4.7k" H 12520 6705 50  0000 L CNN
 F 2 "Resistor_SMD:R_0603_1608Metric" V 12380 6750 50  0001 C CNN
 F 3 "~" H 12450 6750 50  0001 C CNN
@@
 P 12150 7050
 F 0 "R144" V 11943 7050 50  0000 C CNN
-F 1 "100" V 12034 7050 50  0000 C CNN
+F 1 "100R" V 12034 7050 50  0000 C CNN
 F 2 "" V 12080 7050 50  0001 C CNN
 F 3 "~" H 12150 7050 50  0001 C CNN

Commit message: routing
Parts:
- JP1, JP2: footprint (none) -> AR2ISS:SOLDER_JUMPER
- R144: footprint (none) -> Resistor_SMD:R_0603_1608Metric
Changed lines of the file:
@@
 F 0 "JP1" H 4600 3385 50  0000 C CNN
 F 1 "Jumper_NO_Small" H 4600 3294 50  0000 C CNN
-F 2 "" H 4600 3200 50  0001 C CNN
+F 2 "AR2ISS:SOLDER_JUMPER" H 4600 3200 50  0001 C CNN
 F 3 "~" H 4600 3200 50  0001 C CNN
 	1    4600 3200
@@
 F 0 "JP2" H 4600 3485 50  0000 C CNN
 F 1 "Jumper_NO_Small" H 4600 3394 50  0000 C CNN
-F 2 "" H 4600 3300 50  0001 C CNN
+F 2 "AR2ISS:SOLDER_JUMPER" H 4600 3300 50  0001 C CNN
 F 3 "~" H 4600 3300 50  0001 C CNN
 	1    4600 3300
@@
 F 0 "R144" V 11943 7050 50  0000 C CNN
 F 1 "100R" V 12034 7050 50  0000 C CNN
-F 2 "" V 12080 7050 50  0001 C CNN
+F 2 "Resistor_SMD:R_0603_1608Metric" V 12080 7050 50  0001 C CNN
 F 3 "~" H 12150 7050 50  0001 C CNN
 	1    12150 7050

Commit message: ready for jlc
Parts:
- removed JP1, JP2: Jumper_NO_Small, AR2ISS:SOLDER_JUMPER, symbol Device:Jumper_NO_Small
Connections:
- net labels added: +5V
- net labels removed: PWM_DOUT
- wire segments 143 -> 140
- no-connect marks 0 -> 38
Changed lines of the file:
@@
 $Descr A3 16535 11693
 encoding utf-8
-Sheet 21 22
+Sheet 22 22
 Title ""
 Date "2021-04-18"
@@
 Text HLabel 6500 7200 0    50   Input ~ 0
 LD2
-Text HLabel 6550 4700 0    50   Input ~ 0
-CD
-Text HLabel 6550 4800 0    50   Input ~ 0
+Text HLabel 9950 4900 2    50   Input ~ 0
 CE
 Text HLabel 9750 3800 2    50   Input ~ 0
@@
 PWM_DOUT[0..7]
 Text HLabel 2900 2450 0    50   Input ~ 0
-PWM_DOUT
+PWM_DOUT[0..7]
 $Comp
 L AR2ISS:NUCLEO144-H745ZI U2
@@
 Text HLabel 6500 6800 0    50   Input ~ 0
 ADCPWR
-Text HLabel 9850 2300 2    50   Input ~ 0
+Text HLabel 9850 2900 2    50   Input ~ 0
 ADC3V3
 Text Label 9750 3600 0    50   ~ 0
@@
 Wire Wire Line
 	9550 8900 9900 8900
-Text Label 9850 2900 0    50   ~ 0
-PWM_DOUT4
 Text Label 10000 6400 0    50   ~ 0
 PWM_DOUT5
 Wire Wire Line
-	10000 6400 9550 6400
-Wire Wire Line
 	9850 2900 9550 2900
-$Comp
-L Device:Jumper_NO_Small JP1
-U 1 1 60A7645A
-P 4600 3200
-F 0 "JP1" H 4600 3385 50  0000 C CNN
-F 1 "Jumper_NO_Small" H 4600 3294 50  0000 C CNN
-F 2 "AR2ISS:SOLDER_JUMPER" H 4600 3200 50  0001 C CNN
-F 3 "~" H 4600 3200 50  0001 C CNN
-	1    4600 3200
-	1    0    0    -1
-$EndComp
-$Comp
-L Device:Jumper_NO_Small JP2
-U 1 1 60A76AA5
-P 4600 3300
-F 0 "JP2" H 4600 3485 50  0000 C CNN
-F 1 "Jumper_NO_Small" H 4600 3394 50  0000 C CNN
-F 2 "AR2ISS:SOLDER_JUMPER" H 4600 3300 50  0001 C CNN
-F 3 "~" H 4600 3300 50  0001 C CNN
-	1    4600 3300
-	1    0    0    -1
-$EndComp
-Wire Wire Line
-	3650 3300 4500 3300
-Wire Wire Line
-	3650 3200 4500 3200
-Text HLabel 5150 3200 2    50   Input ~ 0
-ENC_A
-Text HLabel 5150 3300 2    50   Input ~ 0
-ENC_B
-Wire Wire Line
-	5150 3300 4700 3300
-Wire Wire Line
-	4700 3200 5150 3200
-Wire Wire Line
-	9850 2300 9550 2300
 Wire Wire Line
 	9850 2600 9550 2600
@@
 	9750 3800 9550 3800
 Wire Wire Line
-	6550 4700 6950 4700
-Wire Wire Line
-	6950 4800 6550 4800
+	9550 4900 9950 4900
 Wire Wire Line
 	6950 7100 6500 7100
@@
 Wire Wire Line
 	9550 8600 9900 8600
+Wire Wire Line
+	3650 3200 4500 3200
+Wire Wire Line
+	3650 3300 4500 3300
+Wire Wire Line
+	9950 6600 9550 6600
+Text HLabel 9950 6600 2    50   Input ~ 0
+CD
+$Comp
+L power:+5V #PWR0147
+U 1 1 60B76364
+P 7550 1700
+F 0 "#PWR0147" H 7550 1550 50  0001 C CNN
+F 1 "+5V" H 7565 1873 50  0000 C CNN
+F 2 "" H 7550 1700 50  0001 C CNN
+F 3 "" H 7550 1700 50  0001 C CNN
+	1    7550 1700
+	1    0    0    -1
+$EndComp
+Wire Wire Line
+	7550 1700 7550 1800
+NoConn ~ 6950 4000
+NoConn ~ 6950 4100
+NoConn ~ 6950 4200
+NoConn ~ 6950 4300
+NoConn ~ 6950 4400
+NoConn ~ 6950 4500
+NoConn ~ 6950 5100
+NoConn ~ 6950 5300
+NoConn ~ 6950 5500
+NoConn ~ 6950 5700
+NoConn ~ 6950 5800
+NoConn ~ 6950 5900
+NoConn ~ 6950 6000
+NoConn ~ 6950 6100
+NoConn ~ 6950 6200
+NoConn ~ 6950 6900
+NoConn ~ 6950 7000
+NoConn ~ 6950 7500
+NoConn ~ 9550 2400
+NoConn ~ 9550 2500
+NoConn ~ 9550 3000
+NoConn ~ 9550 3100
+NoConn ~ 9550 3200
+NoConn ~ 9550 3400
+NoConn ~ 9550 3500
+NoConn ~ 9550 4000
+NoConn ~ 9550 5300
+NoConn ~ 9550 5400
+NoConn ~ 9550 5800
+NoConn ~ 9550 6100
+NoConn ~ 9550 6200
+NoConn ~ 9550 7100
+NoConn ~ 9550 7200
+NoConn ~ 9550 8200
+NoConn ~ 9550 8300
+NoConn ~ 9550 8400
+NoConn ~ 6950 3700
+NoConn ~ 6950 3800
 Wire Bus Line
 	12800 8750 12800 9500
