File: AR2ISS_MainCTL_HW.kicad_pcb (KiCad board)
At the start: 4 copper layers, 200 x 111.5 mm, 297 parts, among them J1 Conn_01x06, J11 Conn_01x02, J12 Conn_01x02, J13 Conn_01x02, J14 Conn_01x02, J15 RJ45_LED, J18 Conn_02x17_Odd_Even, J19 Conn_02x17_Odd_Even, J2 Conn_01x06, J5 Conn_01x08, K1 FINDER-34.51, K2 FINDER-34.51, K3 FINDER-34.51, K4 FINDER-34.51, Q1 BC846, Q2 BC846, Q3 BC846, Q4 BC846, Q5 AO3400A, Q6 APM4953KC, Q7 PMN48XP, U1 MAX3232, U10 MCP23017_SO, U11 LME78_05-1.0, U12 L78033, U13 TSC101B, U14 NCV7608, U15 NCV7608, U16 MCP23017_SO, U17 LM358, U18 LM358, U19 SN75176AD, U2 NUCLEO144-H745ZI, U3 SN75176AD, U4 SN75176AD, U5 SN75176AD, U6 MCP2562-E-SN, U7 MCP23017_SO, U8 TXB0102DCT, U9 74HC164

Commit message: placement
Parts:
- added J16: Conn_01x02, Connector_PinHeader_2.54mm:PinHeader_1x02_P2.54mm_Vertical, F.Cu at (-460.0, -9.91)
- added J17: Conn_01x02, AR2ISS:RM3.5_1x2, F.Cu at (-460.5, -3.17)
- added J22: Conn_01x08, AR2ISS:250-208, F.Cu at (-368.5, -58.8)
- added J23: Conn_01x08, AR2ISS:250-208, F.Cu at (-338.0, -58.8)
- added J24: Conn_02x10_Odd_Even, Connector_IDC:IDC-Header_2x10_P2.54mm_Vertical, F.Cu at (-359.6, -147.7)
- added J25: Conn_02x03_Odd_Even, Connector_IDC:IDC-Header_2x03_P2.54mm_Vertical, F.Cu at (-537.1, -259.5)
- added J26: Conn_01x02, Connector_PinHeader_2.54mm:PinHeader_1x02_P2.54mm_Vertical, F.Cu at (-528.0, -263.3)
- added J3: Conn_01x02, Connector_PinHeader_2.54mm:PinHeader_1x02_P2.54mm_Vertical, F.Cu at (-493.6, -218.4)
- added J6: Conn_02x03_Odd_Even, Connector_PinHeader_2.54mm:PinHeader_2x03_P2.54mm_Vertical, F.Cu at (-496.7, -207.4)
- added J8: DB9_Female, Mouser:23117651, F.Cu at (-519.0, -201.3)
- added J9: Conn_01x02, Connector_PinHeader_2.54mm:PinHeader_1x02_P2.54mm_Vertical, F.Cu at (-492.4, -204.9)
- added L27: L, Inductor_SMD:L_0603_1608Metric, F.Cu at (-720.9, -91.9)
- added L3: 74279266, Inductor_SMD:L_0603_1608Metric, F.Cu at (-484.9, -218.0)
- added L4: 74279266, Inductor_SMD:L_0603_1608Metric, F.Cu at (-484.9, -221.3)
- added L5: 74279266, Inductor_SMD:L_0603_1608Metric, F.Cu at (-483.7, -204.5)
- added L6: 74279266, Inductor_SMD:L_0603_1608Metric, F.Cu at (-483.7, -207.8)
- C16, C17: value 470p -> 1n
- C20, C21: value 1n -> 470p
- D17, D18, D23: footprint Package_TO_SOT_SMD:SOT-23 -> Package_TO_SOT_SMD:SOT-23_Handsoldering
- R38: value 221 -> 120
- R41: value 120 -> 221
- moved C22 624.7 mm to (-261.8, -360.5)
- moved C45 624.7 mm to (-242.9, -410.7)
- moved C49 624.7 mm to (-293.2, -376.1)
- moved L9 624.7 mm to (-257.7, -363.0)
- moved R100 624.7 mm to (-293.2, -378.6)
- moved R101 624.7 mm to (-293.2, -381.1)
- moved R102 624.7 mm to (-289.2, -381.1)
- moved R43 624.7 mm to (-261.8, -363.0)
- moved R44 624.7 mm to (-265.8, -360.5)
- moved R45 624.7 mm to (-265.8, -363.0)
- moved R75 624.7 mm to (-238.9, -410.7)
- moved R76 624.7 mm to (-238.9, -408.2)
- moved R77 624.7 mm to (-242.9, -408.2)
- moved R78 624.7 mm to (-242.9, -405.7)
- moved R99 624.7 mm to (-289.2, -378.6)
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Connections:
- D17 pad 1: /RS232/RS232Filter/A_ext -> /RS232/RS232Filter_1/A_ext
- D17 pad 2: /RS232/RS232Filter/B_ext -> /RS232/RS232Filter_1/B_ext
- D18 pad 1: /RS232/RS232Filter/Y_ext -> /RS232/sheet608DD623/A_ext
- D18 pad 2: /RS232/RS232Filter/Z_ext -> /RS232/sheet608DD623/B_ext
- D24 pad 1: Net-(D24-Pad1) -> /RS422/RS485Tranceiver1/B_in
- D24 pad 2: Net-(D24-Pad2) -> /RS422/RS485Tranceiver1/A_in
- D27 pad 1: Net-(D27-Pad1) -> /RS422/RS485Tranceiver3/B_in
- D27 pad 2: Net-(D27-Pad2) -> /RS422/RS485Tranceiver3/A_in
- D28 pad 1: Net-(D28-Pad1) -> /RS422/RS485Tranceiver4/B_in
- D28 pad 2: Net-(D28-Pad2) -> /RS422/RS485Tranceiver4/A_in
- D29 pad 1: Net-(D29-Pad1) -> /RS422/RS485Tranceiver2/B_in
- D29 pad 2: Net-(D29-Pad2) -> /RS422/RS485Tranceiver2/A_in
- J11 pad 2: Net-(D24-Pad2) -> /RS422/RS485Tranceiver1/A_in
- J12 pad 2: Net-(D27-Pad2) -> /RS422/RS485Tranceiver3/A_in
- J13 pad 2: Net-(D28-Pad2) -> /RS422/RS485Tranceiver4/A_in
- J14 pad 2: Net-(D29-Pad2) -> /RS422/RS485Tranceiver2/A_in
- K1 pad 12: Net-(J1-Pad3) -> Net-(J1-Pad1)
- K1 pad 14: Net-(J1-Pad1) -> Net-(J1-Pad3)
- K2 pad 12: Net-(J1-Pad6) -> Net-(J1-Pad4)
- K2 pad 14: Net-(J1-Pad4) -> Net-(J1-Pad6)
- K3 pad 12: Net-(J2-Pad3) -> Net-(J2-Pad1)
- K3 pad 14: Net-(J2-Pad1) -> Net-(J2-Pad3)
- K4 pad 12: Net-(J2-Pad6) -> Net-(J2-Pad4)
- K4 pad 14: Net-(J2-Pad4) -> Net-(J2-Pad6)
- L10 pad 1: /RS422/RS485Tranceiver1/B_in -> Net-(L10-Pad1)
- L11 pad 1: /RS422/RS485Tranceiver1/A_in -> Net-(L11-Pad1)
- L12 pad 2: Net-(D24-Pad1) -> /RS422/RS485Tranceiver1/B_in
- L13 pad 2: Net-(D24-Pad2) -> /RS422/RS485Tranceiver1/A_in
- L14 pad 1: /RS422/RS485Tranceiver3/B_in -> Net-(L14-Pad1)
- L15 pad 1: /RS422/RS485Tranceiver3/A_in -> Net-(L15-Pad1)
- L16 pad 2: Net-(D27-Pad1) -> /RS422/RS485Tranceiver3/B_in
- L17 pad 2: Net-(D27-Pad2) -> /RS422/RS485Tranceiver3/A_in
- L18 pad 1: /RS422/RS485Tranceiver4/B_in -> Net-(L18-Pad1)
- L19 pad 1: /RS422/RS485Tranceiver4/A_in -> Net-(L19-Pad1)
- L20 pad 2: Net-(D28-Pad1) -> /RS422/RS485Tranceiver4/B_in
- L21 pad 2: Net-(D28-Pad2) -> /RS422/RS485Tranceiver4/A_in
- L22 pad 1: /RS422/RS485Tranceiver2/B_in -> Net-(L22-Pad1)
- L23 pad 1: /RS422/RS485Tranceiver2/A_in -> Net-(L23-Pad1)
- L24 pad 2: Net-(D29-Pad1) -> /RS422/RS485Tranceiver2/B_in
- L25 pad 2: Net-(D29-Pad2) -> /RS422/RS485Tranceiver2/A_in
- R38 pad 1: Net-(C16-Pad1) -> /RS232/sheet608DD623/A_ext
- R38 pad 2: Net-(C20-Pad1) -> Net-(J3-Pad1)
- R39 pad 1: Net-(C17-Pad1) -> Net-(C20-Pad1)
- R39 pad 2: Net-(C21-Pad1) -> Net-(C16-Pad1)
- R40 pad 1: /RS232/RS232Filter/A_ext -> /RS232/RS232Filter_1/A_ext
- R41 pad 1: /RS232/RS232Filter/Y_ext -> Net-(C21-Pad1)
- R41 pad 2: Net-(J10-Pad1) -> Net-(C17-Pad1)
- R48 pad 1: Net-(D24-Pad1) -> /RS422/RS485Tranceiver1/B_in
- R49 pad 2: Net-(D24-Pad1) -> Net-(L10-Pad1)
- R50 pad 1: Net-(D24-Pad1) -> Net-(L10-Pad1)
- R50 pad 2: Net-(D24-Pad2) -> Net-(L11-Pad1)
- R51 pad 1: Net-(D24-Pad2) -> Net-(L11-Pad1)
- R55 pad 1: Net-(D27-Pad1) -> /RS422/RS485Tranceiver3/B_in
- R56 pad 2: Net-(D27-Pad1) -> Net-(L14-Pad1)
- R57 pad 1: Net-(D27-Pad1) -> Net-(L14-Pad1)
- R57 pad 2: Net-(D27-Pad2) -> Net-(L15-Pad1)
- R58 pad 1: Net-(D27-Pad2) -> Net-(L15-Pad1)
- R62 pad 1: Net-(D28-Pad1) -> /RS422/RS485Tranceiver4/B_in
- R63 pad 2: Net-(D28-Pad1) -> Net-(L18-Pad1)
- R64 pad 1: Net-(D28-Pad1) -> Net-(L18-Pad1)
- R64 pad 2: Net-(D28-Pad2) -> Net-(L19-Pad1)
- R65 pad 1: Net-(D28-Pad2) -> Net-(L19-Pad1)
- R69 pad 1: Net-(D29-Pad1) -> /RS422/RS485Tranceiver2/B_in
- R70 pad 2: Net-(D29-Pad1) -> Net-(L22-Pad1)
- R71 pad 1: Net-(D29-Pad1) -> Net-(L22-Pad1)
- R71 pad 2: Net-(D29-Pad2) -> Net-(L23-Pad1)
- R72 pad 1: Net-(D29-Pad2) -> Net-(L23-Pad1)
- U1 pad 13: /RS232/RS232Filter/Z_ext -> /RS232/sheet608DD623/B_int
- U1 pad 14: /RS232/RS232Filter/B_ext -> /RS232/RS232Filter_1/B_int
- U1 pad 7: /RS232/RS232Filter/A_ext -> /RS232/RS232Filter_1/A_int
- U1 pad 8: /RS232/RS232Filter/Y_ext -> /RS232/sheet608DD623/A_int
- U19 pad 6: Net-(D29-Pad2) -> Net-(L23-Pad1)
- U19 pad 7: Net-(D29-Pad1) -> Net-(L22-Pad1)
- U3 pad 6: Net-(D24-Pad2) -> Net-(L11-Pad1)
- U3 pad 7: Net-(D24-Pad1) -> Net-(L10-Pad1)
- U4 pad 6: Net-(D27-Pad2) -> Net-(L15-Pad1)
- U4 pad 7: Net-(D27-Pad1) -> Net-(L14-Pad1)
- U5 pad 6: Net-(D28-Pad2) -> Net-(L19-Pad1)
- U5 pad 7: Net-(D28-Pad1) -> Net-(L18-Pad1)
Routing:
- net /LCD/BTN9: track 0.00 -> 49.0 mm
- net /LCD/BTN11: track 0.00 -> 48.3 mm
- net /LCD/BTN8: track 0.00 -> 46.5 mm
- net /LCD/BTN10: track 0.00 -> 45.9 mm
- net /LCD/BTN3: track 0.00 -> 42.6 mm
- net /LCD/BTN12: track 0.00 -> 41.0 mm
- net /LCD/BTN4: track 0.00 -> 40.7 mm
- net /LCD/BTN1: track 0.00 -> 40.3 mm
- net /LCD/BTN2: track 0.00 -> 38.3 mm
- net +12V: track 39.3 -> 74.9 mm
- net /LCD/BTN0: track 0.00 -> 33.9 mm
- net GND: track 124.9 -> 155.1 mm, vias 25 -> 54
- net /RS232/RS232Filter_1/B_ext: track 0.00 -> 28.0 mm, vias 0 -> 1
- net /IOExpander/IO1: track 0.00 -> 25.8 mm
- net /IOExpander/IO2: track 0.00 -> 25.7 mm
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Other:
- board size 200 x 111.5 mm -> 200.7 x 111.8 mm

Commit message: add TLE5602
Parts:
- removed Q5: AO3400A, Package_TO_SOT_SMD:SOT-23
- removed Q6: APM4953KC, Package_SO:SO-8_5.3x6.2mm_P1.27mm
- added C54: 100n, Capacitor_SMD:C_0603_1608Metric, F.Cu at (-213.2, -137.8)
- added C75: 100n, Capacitor_SMD:C_0603_1608Metric, F.Cu at (-209.2, -137.8)
- added D19: LED, LED_SMD:LED_0603_1608Metric, F.Cu at (-213.1, -140.3)
- added D20: D_Zener, Diode_SMD:D_SOD-123, F.Cu at (-332.3, -201.0)
- added D21: D_TVS, Diode_SMD:D_SMA-SMB_Universal_Handsoldering, F.Cu at (-289.8, -150.6)
- added D26: D_Schottky, Diode_SMD:D_SOD-123, F.Cu at (-332.3, -191.9)
- added D30: LED, LED_SMD:LED_0603_1608Metric, F.Cu at (-209.1, -140.3)
- added D31: BZX84Cxx, Diode_SMD:D_SOT-23_ANK, F.Cu at (-217.4, -139.4)
- added D32: BZX84Cxx, Diode_SMD:D_SOT-23_ANK, F.Cu at (-217.4, -134.8)
- added J4: Conn_01x02, AR2ISS:250-202, F.Cu at (-270.7, -142.7)
- added L1: 10u, Inductor_SMD:L_0603_1608Metric, F.Cu at (-309.5, -199.0)
- added L2: 10u, Inductor_SMD:L_0603_1608Metric, F.Cu at (-305.5, -199.0)
- added L7: 10u, Inductor_SMD:L_0603_1608Metric, F.Cu at (-309.5, -206.9)
- added L8: 10u, Inductor_SMD:L_0603_1608Metric, F.Cu at (-305.5, -206.9)
- added R104: NB, Resistor_SMD:R_0603_1608Metric, F.Cu at (-327.4, -198.9)
- added R141: 15k, Resistor_SMD:R_0603_1608Metric, F.Cu at (-209.2, -135.3)
- added R142: 1k, Resistor_SMD:R_0603_1608Metric, F.Cu at (-205.2, -137.8)
- added R143: 10meg, Resistor_SMD:R_0603_1608Metric, F.Cu at (-209.2, -132.8)
- added R42: 470, Resistor_SMD:R_0603_1608Metric, F.Cu at (-283.0, -163.3)
- J17: footprint AR2ISS:RM3.5_1x2 -> AR2ISS:250-202
- J8: footprint Mouser:23117651 -> AR2ISS:L177TSEH09SOL2RM8
- R105: value 6.2k -> 82k
- R106, R110: value 1k -> 10k
- R108: value 10k -> 1.5k
- R109: value 100k -> 470
- U14, U15: value NCV7608 -> TLE75602-ESH; footprint Package_SO:SOIC-28W_7.5x17.9mm_P1.27mm -> AR2ISS:Infineon_PG-TSDSO-24-21
- moved J25 474.5 mm to (-138.3, -2.36), turned to 180 degrees
- moved J26 463.7 mm to (-147.3, 1.44), turned to 180 degrees
- moved F2 412.2 mm to (-352.0, -63.9), turned to 180 degrees
- moved L27 373.5 mm to (-351.3, -146.5), turned to 90 degrees
- moved J3 370.9 mm to (-179.7, -20.8)
- moved D18 362.9 mm to (-185.2, -20.7)
- moved C21 357.3 mm to (-183.4, -26.9), turned to 180 degrees
- moved R38 357.1 mm to (-187.4, -26.8)
- moved C17 356.6 mm to (-184.0, -24.3)
- moved C16 356.3 mm to (-179.4, -26.9)
- moved L3 354.5 mm to (-188.0, -24.3), turned to 180 degrees
- moved L4 353.6 mm to (-194.5, -19.7), turned to 180 degrees
- moved C20 353.5 mm to (-190.5, -19.7), turned to 180 degrees
- moved J6 352.9 mm to (-178.7, -54.4), turned to 90 degrees
- moved R39 349.2 mm to (-192.0, -22.2), turned to 180 degrees
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Connections:
- net Net-(U2-Pad118) renamed /Controller/PWM_DOUT2
- net Net-(U2-Pad120) renamed /Controller/PWM_DOUT3
- net Net-(U2-Pad123) renamed /Controller/PWM_DOUT1
- net Net-(U2-Pad127) renamed /Controller/PWM_DOUT0
- net Net-(U2-Pad3) renamed /SDCard/CLK
- net Net-(U2-Pad85) renamed /Controller/PWM_DOUT4
- net Net-(U2-Pad90) renamed /Controller/SDA_ext
- net Net-(U2-Pad91) renamed /Controller/PWM_DOUT5
- net Net-(U2-Pad97) renamed /Controller/SCL_ext
- C50 pad 1: Net-(C50-Pad1) -> +12V
- C52 pad 1: Net-(C50-Pad1) -> +12V
- C57 pad 1: /PowerSupply/ADC12V -> /Controller/ADC12V
- C61 pad 2: Net-(C61-Pad2) -> +12V
- C65 pad 1: +12V -> +12VA
- C69 pad 1: Net-(C69-Pad1) -> /Controller/NRST
- D22 pad 1: Net-(D22-Pad1) -> /Controller/ONEWIRE
- D22 pad 2: Net-(D22-Pad2) -> GND
- D25 pad 1: /PowerSupply/ADC12V -> /Controller/ADC12V
- F1 pad 2: +12V -> Net-(F1-Pad2)
- F2 pad 1: Net-(C61-Pad1) -> +12VA
- J22 pad 7: +12V -> Net-(J22-Pad7)
- J22 pad 8: GND -> Net-(J22-Pad8)
- J23 pad 7: +12V -> Net-(J23-Pad7)
- J23 pad 8: GND -> Net-(J23-Pad8)
- J24 pad 10: Net-(J24-Pad10) -> /DOut/IO7
- J24 pad 11: Net-(J24-Pad11) -> /DOut/IO8
- J24 pad 12: Net-(J24-Pad12) -> /DOut/IO9
- J24 pad 13: Net-(J24-Pad13) -> /DOut/IO10
- J24 pad 14: Net-(J24-Pad14) -> /DOut/IO11
- J24 pad 15: Net-(J24-Pad15) -> /DOut/IO12
- J24 pad 16: Net-(J24-Pad16) -> /DOut/IO13
- J24 pad 17: Net-(J24-Pad17) -> /DOut/IO14
- J24 pad 18: Net-(J24-Pad18) -> /DOut/IO15
- J24 pad 2: Net-(J24-Pad2) -> Net-(J24-Pad1)
- J24 pad 3: Net-(J24-Pad3) -> /DOut/IO0
- J24 pad 4: Net-(J24-Pad4) -> /DOut/IO1
- J24 pad 5: Net-(J24-Pad5) -> /DOut/IO2
- J24 pad 6: Net-(J24-Pad6) -> /DOut/IO3
- J24 pad 7: Net-(J24-Pad7) -> /DOut/IO4
- J24 pad 8: Net-(J24-Pad8) -> /DOut/IO5
- J24 pad 9: Net-(J24-Pad9) -> /DOut/IO6
- J25 pad 3: Net-(C69-Pad1) -> /Controller/NRST
- J26 pad 1: /Controller/ONEWIRE -> Net-(J26-Pad1)
- Q7 pad 4: Net-(C50-Pad1) -> Net-(C61-Pad1)
- R105 pad 2: /PowerSupply/ADC12V -> /Controller/ADC12V
- R106 pad 1: /PowerSupply/ADC12V -> /Controller/ADC12V
- R107 pad 1: Net-(C61-Pad2) -> +12V
- R108 pad 1: Net-(C61-Pad2) -> +12V
- R108 pad 2: Net-(Q6-Pad2) -> Net-(D19-Pad2)
- R109 pad 1: /PowerSupply/PREAMP_ON -> +5V
- R109 pad 2: GND -> Net-(D30-Pad2)
- R110 pad 1: Net-(Q6-Pad2) -> +5V
- R110 pad 2: Net-(Q5-Pad3) -> /Controller/ADC5V
- R120 pad 2: /Controller/EN2 -> /Controller/EN1
- R126 pad 2: Net-(C69-Pad1) -> /Controller/NRST
- R127 pad 2: /Controller/ONEWIRE -> Net-(J26-Pad1)
- R128 pad 2: /SDCard/MISO -> /SDCard/D0
- R129 pad 2: /SDCard/#CS -> /SDCard/#CD
- R130 pad 2: /SDCard/MOSI -> /SDCard/CMD
- R59 pad 1: GND -> /RS422/RS485Tranceiver1/MODE
- U1 pad 10: /RS232/T2IN -> /Controller/COM_TX2
- U1 pad 11: /RS232/T1IN -> /Controller/COM_TX1
- U1 pad 12: /RS232/R1OUT -> /Controller/COM_RX1
- U1 pad 9: /RS232/R2OUT -> /Controller/COM_RX2
- U11 pad 1: Net-(C50-Pad1) -> +12V
- U12 pad 1: +5V -> Net-(R104-Pad1)
- U13 pad 1: /PowerSupply/ADCPWR -> /Controller/ADCPWR
- U13 pad 3: Net-(C61-Pad2) -> +12V
- U14 pad 1: +12V -> /Controller/#CS1
- U14 pad 10: GND -> Net-(J22-Pad3)
- U14 pad 12: GND -> +12VA
- U14 pad 13: Net-(J22-Pad5) -> +12VA
- U14 pad 14: +12V -> Net-(J22-Pad6)
- U14 pad 15: +12V -> Net-(J22-Pad4)
- U14 pad 16: Net-(J22-Pad6) -> +12VA
- U14 pad 17: GND -> Net-(J22-Pad2)
- U14 pad 18: Net-(J22-Pad6) -> +12VA
- U14 pad 19: /Controller/EN1 -> Net-(J22-Pad8)
- U14 pad 2: Net-(J22-Pad2) -> Net-(R113-Pad1)
- U14 pad 20: /MESAOut/PWM_DOUT0 -> +12VA
- U14 pad 21: /MESAOut/PWM_DOUT1 -> /Controller/EN1
- U14 pad 22: /MESAOut/PWM_DOUT2 -> /MESAOut/PWM_DOUT1
- U14 pad 23: /MESAOut/PWM_DOUT3 -> /MESAOut/PWM_DOUT0
- U14 pad 24: +12V -> +3V3
- U14 pad 25: +12V -> GND
- U14 pad 3: Net-(J22-Pad1) -> Net-(R114-Pad1)
- U14 pad 4: +12V -> Net-(R115-Pad1)
- U14 pad 5: /Controller/#CS1 -> GND
- U14 pad 6: Net-(R113-Pad1) -> Net-(J22-Pad7)
- U14 pad 7: Net-(R114-Pad1) -> +12VA
- U14 pad 8: +3V3 -> Net-(J22-Pad1)
- U14 pad 9: Net-(R115-Pad1) -> +12VA
- U15 pad 1: +12V -> /Controller/#CS2
- U15 pad 10: GND -> Net-(J23-Pad3)
- U15 pad 12: GND -> +12VA
- U15 pad 13: Net-(J23-Pad5) -> +12VA
- U15 pad 14: +12V -> Net-(J23-Pad6)
- U15 pad 15: +12V -> Net-(J23-Pad4)
- U15 pad 16: Net-(J23-Pad6) -> +12VA
- U15 pad 17: GND -> Net-(J23-Pad2)
- U15 pad 18: Net-(J23-Pad6) -> +12VA
- U15 pad 19: /Controller/EN2 -> Net-(J23-Pad8)
- U15 pad 2: Net-(J23-Pad2) -> Net-(R117-Pad1)
- U15 pad 20: /MESAOut/PWM_DOUT4 -> +12VA
- U15 pad 21: /MESAOut/PWM_DOUT5 -> /Controller/EN1
- U15 pad 22: /MESAOut/PWM_DOUT6 -> /MESAOut/PWM_DOUT3
- U15 pad 23: /MESAOut/PWM_DOUT7 -> /MESAOut/PWM_DOUT2
- U15 pad 24: +12V -> +3V3
- U15 pad 25: +12V -> GND
- U15 pad 3: Net-(J23-Pad1) -> Net-(R118-Pad1)
- U15 pad 4: +12V -> Net-(R119-Pad1)
- U15 pad 5: /Controller/#CS2 -> GND
- U15 pad 6: Net-(R117-Pad1) -> Net-(J23-Pad7)
- U15 pad 7: Net-(R118-Pad1) -> +12VA
- U15 pad 8: +3V3 -> Net-(J23-Pad1)
- U15 pad 9: Net-(R119-Pad1) -> +12VA
- U16 pad 1: /DOut/sheet60ADF1E9/IO0 -> /DOut/IO0
- U16 pad 2: /DOut/sheet60ADF1E9/IO1 -> /DOut/IO1
- U16 pad 21: /DOut/sheet60ADF1E9/IO8 -> /DOut/IO8
- U16 pad 22: /DOut/sheet60ADF1E9/IO9 -> /DOut/IO9
- U16 pad 23: /DOut/sheet60ADF1E9/IO10 -> /DOut/IO10
- U16 pad 24: /DOut/sheet60ADF1E9/IO11 -> /DOut/IO11
- U16 pad 25: /DOut/sheet60ADF1E9/IO12 -> /DOut/IO12
- U16 pad 26: /DOut/sheet60ADF1E9/IO13 -> /DOut/IO13
- U16 pad 27: /DOut/sheet60ADF1E9/IO14 -> /DOut/IO14
- U16 pad 28: /DOut/sheet60ADF1E9/IO15 -> /DOut/IO15
- U16 pad 3: /DOut/sheet60ADF1E9/IO2 -> /DOut/IO2
- U16 pad 4: /DOut/sheet60ADF1E9/IO3 -> /DOut/IO3
- U16 pad 5: /DOut/sheet60ADF1E9/IO4 -> /DOut/IO4
- U16 pad 6: /DOut/sheet60ADF1E9/IO5 -> /DOut/IO5
- U16 pad 7: /DOut/sheet60ADF1E9/IO6 -> /DOut/IO6
- U16 pad 8: /DOut/sheet60ADF1E9/IO7 -> /DOut/IO7
- U2 pad 1: Net-(U2-Pad1) -> /Controller/SCLK
- U2 pad 103: Net-(U2-Pad103) -> /Controller/SWO
- U2 pad 105: Net-(U2-Pad105) -> /Controller/COM_RX2
- U2 pad 109: Net-(U2-Pad109) -> /Controller/ADC5V
- U2 pad 11: Net-(U2-Pad11) -> /ADIn/DA_IN_LL3
- U2 pad 112: Net-(U2-Pad112) -> /Controller/COM_TX1
- U2 pad 113: Net-(U2-Pad113) -> /Controller/EN1
- U2 pad 114: Net-(U2-Pad114) -> /ADIn/DA_IN_LL4
- U2 pad 115: Net-(U2-Pad115) -> /Controller/#CS2
- U2 pad 116: Net-(U2-Pad116) -> /Controller/COM_RX1
- U2 pad 117: Net-(U2-Pad117) -> /Controller/#CS1
- U2 pad 122: Net-(U2-Pad122) -> /Controller/LD1
- U2 pad 124: Net-(U2-Pad124) -> /Controller/ENC_A
- U2 pad 125: Net-(U2-Pad125) -> /SDCard/#CD
- U2 pad 128: Net-(U2-Pad128) -> /Controller/ENC_B
- U2 pad 13: Net-(U2-Pad13) -> /Controller/SWDIO
- U2 pad 132: Net-(U2-Pad132) -> /Controller/LD2
- U2 pad 133: Net-(U2-Pad133) -> /Controller/TX2
- U2 pad 134: Net-(U2-Pad134) -> /Controller/ADCPWR
- U2 pad 138: Net-(U2-Pad138) -> /Controller/CE
- U2 pad 139: Net-(U2-Pad139) -> /Controller/CD
- U2 pad 14: Net-(U2-Pad14) -> /Controller/NRST
- U2 pad 15: Net-(U2-Pad15) -> /Controller/SWCLK
- U2 pad 17: Net-(U2-Pad17) -> /Controller/Backlight
- U2 pad 2: Net-(U2-Pad2) -> /Controller/MISO
- U2 pad 21: Net-(U2-Pad21) -> /Controller/SDA
- U2 pad 28: Net-(U2-Pad28) -> /Controller/ADC3V3
- U2 pad 32: Net-(U2-Pad32) -> /AOut/DAC1
- U2 pad 35: Net-(U2-Pad35) -> /ADIn/DA_IN_LL0
- U2 pad 37: Net-(U2-Pad37) -> /ADIn/DA_IN_LL1
- U2 pad 38: Net-(U2-Pad38) -> /ADIn/DA_IN_LL7
- U2 pad 4: Net-(U2-Pad4) -> /SDCard/CMD
- U2 pad 40: Net-(U2-Pad40) -> /Controller/DisplayCLK
- U2 pad 41: Net-(U2-Pad41) -> /Controller/TX
- U2 pad 43: Net-(U2-Pad43) -> /Controller/RX
- U2 pad 47: Net-(U2-Pad47) -> /Controller/REL1
- U2 pad 48: Net-(U2-Pad48) -> /Controller/REL2
- U2 pad 50: Net-(U2-Pad50) -> /Controller/REL3
- U2 pad 54: Net-(U2-Pad54) -> /ADIn/DA_IN_LL5
- U2 pad 55: Net-(U2-Pad55) -> /CAN/FDCAN_TX
- U2 pad 56: Net-(U2-Pad56) -> /ADIn/DA_IN_LL2
- U2 pad 57: Net-(U2-Pad57) -> /CAN/FDCAN_RX
- U2 pad 62: Net-(U2-Pad62) -> /Controller/REL4
- U2 pad 63: Net-(U2-Pad63) -> /Controller/RX2
- U2 pad 74: Net-(U2-Pad74) -> /SDCard/D0
- U2 pad 75: Net-(U2-Pad75) -> /Controller/SCL
- U2 pad 76: Net-(U2-Pad76) -> /Controller/ONEWIRE
- U2 pad 83: Net-(U2-Pad83) -> /AOut/DAC2
- U2 pad 89: Net-(U2-Pad89) -> /Controller/COM_TX2
- U2 pad 9: Net-(U2-Pad9) -> /ADIn/DA_IN_LL6
- U2 pad 94: Net-(U2-Pad94) -> /Controller/MOSI
- U2 pad 96: Net-(U2-Pad96) -> /Controller/ADC12V
- U2 pad 98: Net-(U2-Pad98) -> /Controller/DisplayData
- U4 pad 1: /RS422/PTT1 -> /Controller/TX2
- U4 pad 3: /RS422/PTT1 -> /Controller/TX2
- U5 pad 1: /RS422/PTT2 -> /Controller/RX2
- U5 pad 3: /RS422/PTT2 -> /Controller/RX2
Routing:
- net Net-(J22-Pad7): track 0.00 -> 68.6 mm
- net Net-(J22-Pad2): track 0.00 -> 56.3 mm
- net /ADIn/DA_IN_LL1: track 0.00 -> 52.8 mm
- net Net-(J22-Pad4): track 0.00 -> 46.6 mm
- net /ADIn/DA_IN_LL0: track 0.00 -> 45.8 mm
- net /ADIn/DA_IN_0: track 18.2 -> 60.6 mm
- net Net-(J22-Pad8): track 0.00 -> 41.8 mm
- net /ADIn/DA_IN_1: track 22.7 -> 63.5 mm
- net /RS422/RS485Tranceiver1/MODE: track 42.5 -> 2.70 mm, vias 10 -> 6
- net /ADIn/DA_IN_2: track 19.2 -> 55.9 mm
- net /ADIn/DA_IN_3: track 23.1 -> 58.3 mm
- net /ADIn/DA_IN_5: track 22.6 -> 57.8 mm
- net /ADIn/DA_IN_4: track 17.8 -> 52.3 mm
- net Net-(J23-Pad5): track 0.00 -> 34.4 mm
- net Net-(J22-Pad6): track 0.00 -> 34.4 mm
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- added copper zone on In1.Cu, net GND

Commit message: routing
Parts:
- D25, D31, D32: value BZX84Cxx -> BZX84C3V6,215
- D26: value D_Schottky -> BAT54W-HG3-08
- R103, R52, R59, R66: value 3k -> 4.7k
- R111, R112, R116, R120: value 100k -> NB
- R127: value 4k7 -> 4.7k
- R49, R51, R56, R58, R63, R65, R70, R72: value 10k -> NB
- R50, R57, R64, R71: value 1k -> NB
- U19, U3, U4, U5: value SN75176AD -> SP3485EN-L/TR
- U8: value TXB0102DCT -> NTB0102DP
- moved J25 361.4 mm to (-484.2, -107.1), turned to 270 degrees
- moved L2 119.2 mm to (-303.7, -79.8), turned to 90 degrees
- moved L1 116.2 mm to (-303.7, -83.0), turned to 270 degrees
- moved C18 108.6 mm to (-301.4, -84.1)
- moved R36 108.6 mm to (-301.4, -82.5)
- moved J9 108.5 mm to (-288.4, -82.6)
- moved R40 108.5 mm to (-292.2, -84.2)
- moved C14 108.5 mm to (-298.8, -83.0)
- moved C15 108.5 mm to (-298.8, -79.7)
- moved D17 108.5 mm to (-293.2, -81.4)
- moved J6 108.5 mm to (-284.1, -80.1)
- moved L5 108.5 mm to (-297.0, -83.0)
- moved L6 108.5 mm to (-297.0, -79.7)
- moved C19 108.4 mm to (-301.4, -78.7)
- moved R37 108.4 mm to (-301.4, -80.3)
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Connections:
- J15 pad 13: Net-(J15-Pad13) -> Net-(C22-Pad2)
- R49 pad 2: Net-(L10-Pad1) -> Net-(L11-Pad1)
- R50 pad 1: Net-(L10-Pad1) -> Net-(L11-Pad1)
- R50 pad 2: Net-(L11-Pad1) -> Net-(L10-Pad1)
- R51 pad 1: Net-(L11-Pad1) -> Net-(L10-Pad1)
- R56 pad 2: Net-(L14-Pad1) -> Net-(L15-Pad1)
- R57 pad 1: Net-(L14-Pad1) -> Net-(L15-Pad1)
- R57 pad 2: Net-(L15-Pad1) -> Net-(L14-Pad1)
- R58 pad 1: Net-(L15-Pad1) -> Net-(L14-Pad1)
- R63 pad 2: Net-(L18-Pad1) -> Net-(L19-Pad1)
- R64 pad 1: Net-(L18-Pad1) -> Net-(L19-Pad1)
- R64 pad 2: Net-(L19-Pad1) -> Net-(L18-Pad1)
- R65 pad 1: Net-(L19-Pad1) -> Net-(L18-Pad1)
- R70 pad 2: Net-(L22-Pad1) -> Net-(L23-Pad1)
- R71 pad 1: Net-(L22-Pad1) -> Net-(L23-Pad1)
- R71 pad 2: Net-(L23-Pad1) -> Net-(L22-Pad1)
- R72 pad 1: Net-(L23-Pad1) -> Net-(L22-Pad1)
- U19 pad 3: /Controller/RX -> /RS422/RS485Tranceiver2/DE1
- U19 pad 4: /RS422/RS485Tranceiver2/DE1 -> /Controller/RX
- U3 pad 3: /Controller/TX -> /RS422/RS485Tranceiver1/DE1
- U3 pad 4: /RS422/RS485Tranceiver1/DE1 -> /Controller/TX
- U4 pad 3: /Controller/TX2 -> /RS422/RS485Tranceiver3/DE1
- U4 pad 4: /RS422/RS485Tranceiver3/DE1 -> /Controller/TX2
- U5 pad 3: /Controller/RX2 -> /RS422/RS485Tranceiver4/DE1
- U5 pad 4: /RS422/RS485Tranceiver4/DE1 -> /Controller/RX2
Routing:
- net +12VA: track 0.00 -> 98.4 mm, vias 0 -> 12
- net Net-(J23-Pad7): track 0.00 -> 66.2 mm
- net Net-(D23-Pad1): track 3.51 -> 63.5 mm, vias 0 -> 1
- net Net-(D23-Pad2): track 9.15 -> 66.9 mm, vias 0 -> 1
- net Net-(J23-Pad8): track 0.00 -> 50.0 mm, vias 0 -> 1
- net /ADIn/DA_IN_LL4: track 0.00 -> 47.0 mm
- net /ADIn/DA_IN_LL5: track 0.00 -> 44.2 mm, vias 0 -> 1
- net GND: track 153.6 -> 197.0 mm, vias 44 -> 52
- net /RS422/RS485Tranceiver1/B_in: track 5.69 -> 45.4 mm, vias 0 -> 1
- net /ADIn/DA_IN_LL3: track 0.00 -> 38.3 mm, vias 0 -> 2
- net Net-(J23-Pad6): track 0.00 -> 37.4 mm
- net /RS422/RS485Tranceiver2/B_in: track 5.69 -> 41.1 mm
- net /ADIn/DA_IN_LL6: track 0.00 -> 34.6 mm, vias 0 -> 1
- net /CAN/FDCAN_TX: track 0.00 -> 32.7 mm, vias 0 -> 1
- net Net-(J23-Pad3): track 3.19 -> 34.4 mm
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- added copper zone on In2.Cu, net +3V3

Commit message: routing
Parts:
- added J28: Conn_01x04, AR2ISS:250-204, F.Cu at (-324.0, -166.8)
- added JP1: Jumper_NO_Small, AR2ISS:SOLDER_JUMPER, F.Cu at (-408.4, -10.2)
- added JP2: Jumper_NO_Small, AR2ISS:SOLDER_JUMPER, F.Cu at (-412.8, -27.3)
- added R144: 100R, Resistor_SMD:R_0603_1608Metric, F.Cu at (-407.0, -25.1)
- moved C71 173.1 mm to (-355.5, -181.8)
- moved C72 173.1 mm to (-355.5, -179.3)
- moved C73 173.1 mm to (-351.5, -181.8)
- moved C74 173.1 mm to (-342.6, -185.7)
- moved R133 173.1 mm to (-343.4, -180.7)
- moved R134 173.1 mm to (-359.5, -181.8)
- moved R135 173.1 mm to (-347.4, -179.3)
- moved R136 173.1 mm to (-342.6, -183.2)
- moved R137 173.1 mm to (-351.5, -179.3)
- moved R138 173.1 mm to (-347.4, -181.8)
- moved R140 173.1 mm to (-359.5, -179.3)
- moved R139 173.1 mm to (-342.6, -188.2)
- moved U17 173.1 mm to (-348.8, -186.3)
- moved U18 173.1 mm to (-357.3, -186.3)
Connections:
- net /RS422/RS485Tranceiver1/MODE renamed /RS422/VCC_RS422

Commit message: placement, routing
Parts:
- removed R121, R122, R123, R124: R, Resistor_SMD:R_0603_1608Metric
- added J27: Micro_SD_Card, Connector_Card:microSD_HC_Wuerth_693072010801, F.Cu at (-413.2, -194.0)
- added J7: Conn_01x03, Connector_PinHeader_2.54mm:PinHeader_1x03_P2.54mm_Vertical, F.Cu at (-278.3, -26.8)
- R100, R102, R78: value R -> 0R
- R101, R76, R77, R99: value R -> NB
- R75: value R -> 4.7k
- moved R125 263.4 mm to (-319.6, 0.72)
- moved BT1 257.2 mm to (-321.9, -4.87)
- moved C68 241.9 mm to (-314.4, 0.34)
- moved C69 235.9 mm to (-357.9, -80.9), turned to 180 degrees
- moved R127 226.2 mm to (-338.0, -17.8)
- moved D22 223.9 mm to (-339.3, -23.9), turned to 90 degrees
- moved R129 206.1 mm to (-413.2, -180.4)
- moved R130 206.1 mm to (-417.2, -180.4)
- moved R131 206.1 mm to (-409.2, -180.4)
- moved C70 206.1 mm to (-417.2, -177.9)
- moved R128 206.1 mm to (-413.2, -177.9)
- moved R132 206.1 mm to (-409.2, -177.9)
- moved D26 192.4 mm to (-326.2, 0.47)
- moved J26 187.8 mm to (-333.6, -22.9)
- moved L8 184.4 mm to (-311.2, -22.6)
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Connections:
- net Net-(R101-Pad2) renamed /IOExpander2/A1
- R100 pad 1: Net-(R100-Pad1) -> /IOExpander/A1
- R75 pad 2: Net-(R75-Pad2) -> /IOExpander/A0
- R76 pad 1: Net-(R75-Pad2) -> /IOExpander/A0
- R77 pad 2: Net-(R77-Pad2) -> /IOExpander2/A0
- R78 pad 1: Net-(R77-Pad2) -> /IOExpander2/A0
- R99 pad 2: Net-(R100-Pad1) -> /IOExpander/A1
- U10 pad 15: GND -> /IOExpander2/A0
- U10 pad 17: Net-(R100-Pad1) -> GND
- U16 pad 15: GND -> /DOut/sheet60ADF1E9/A0
- U16 pad 16: Net-(R123-Pad2) -> /DOut/sheet60ADF1E9/A1
- U16 pad 17: Net-(R121-Pad2) -> /DOut/sheet60ADF1E9/A2
- U17 pad 5: Net-(C74-Pad1) -> Net-(R137-Pad1)
- U17 pad 6: Net-(R136-Pad1) -> Net-(J28-Pad1)
- U17 pad 7: Net-(R138-Pad1) -> Net-(J28-Pad1)
- U18 pad 1: Net-(J28-Pad1) -> Net-(R138-Pad1)
- U18 pad 2: Net-(J28-Pad1) -> Net-(R136-Pad1)
- U18 pad 3: Net-(R137-Pad1) -> Net-(C74-Pad1)
- U7 pad 15: GND -> /IOExpander/A0
- U7 pad 16: Net-(R77-Pad2) -> /IOExpander/A1
- U7 pad 17: Net-(R75-Pad2) -> GND
Routing:
- net +12V: track 101.3 -> 315.5 mm, vias 0 -> 1
- net /Controller/REL2: track 0.00 -> 156.3 mm, vias 0 -> 3
- net /Controller/REL1: track 11.3 -> 163.7 mm, vias 0 -> 3
- net /Controller/REL4: track 0.00 -> 146.4 mm, vias 0 -> 3
- net /Controller/REL3: track 0.00 -> 144.2 mm, vias 0 -> 3
- net /AOut/DAC1: track 0.00 -> 85.6 mm, vias 0 -> 1
- net /Controller/COM_TX2: track 0.00 -> 78.6 mm, vias 0 -> 1
- net /Controller/LD2: track 0.00 -> 65.5 mm
- net /Controller/TX: track 0.00 -> 59.9 mm, vias 0 -> 2
- net /ADIn/DA_IN_LL2: track 0.00 -> 58.1 mm, vias 0 -> 2
- net /Controller/COM_TX1: track 0.00 -> 58.1 mm, vias 0 -> 1
- net /Controller/COM_RX1: track 0.00 -> 58.0 mm, vias 0 -> 1
- net /Controller/COM_RX2: track 0.00 -> 57.5 mm, vias 0 -> 1
- net GND: track 197.0 -> 252.9 mm, vias 52 -> 68
- net /RS422/VCC_RS422: track 8.91 -> 64.7 mm, vias 0 -> 4
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Other:
- board text added: "adc spannungen"
- board text added: "batt"
- board text added: "onewire"
- board text added: "rs232 2"

Commit message: Update AR2ISS_MainCTL_HW.kicad_pcb
Parts:
- moved D25 138.5 mm to (-331.6, -143.7), turned to 90 degrees
- moved R142 137.7 mm to (-342.7, -143.4), turned to 270 degrees
- moved R105 136.5 mm to (-334.6, -143.4), turned to 270 degrees
- moved R106 135.8 mm to (-334.6, -140.0), turned to 270 degrees
- moved C57 134.5 mm to (-332.7, -140.0), turned to 270 degrees
- moved R143 133.7 mm to (-342.7, -140.0), turned to 270 degrees
- moved C75 131.4 mm to (-340.5, -140.0), turned to 270 degrees
- moved R108 123.6 mm to (-336.5, -143.4), turned to 270 degrees
- moved R109 123.6 mm to (-328.6, -143.4), turned to 270 degrees
- moved D19 123.3 mm to (-336.5, -140.0), turned to 90 degrees
- moved D32 122.4 mm to (-339.5, -143.7), turned to 90 degrees
- moved D30 119.5 mm to (-328.6, -140.0), turned to 90 degrees
- moved R141 117.5 mm to (-326.6, -140.0), turned to 270 degrees
- moved R110 113.9 mm to (-326.6, -143.4), turned to 270 degrees
- moved C54 111.4 mm to (-324.5, -140.0), turned to 270 degrees
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Routing:
- net /Controller/SWCLK: track 0.00 -> 87.7 mm
- net /Controller/SWDIO: track 0.00 -> 79.4 mm
- net GND: track 252.9 -> 288.2 mm, vias 68 -> 71
- net +5V: track 22.9 -> 46.5 mm
- net /Controller/ADC5V: track 0.00 -> 21.4 mm, vias 0 -> 1
- net /Controller/ADC12V: track 0.00 -> 20.2 mm, vias 0 -> 1
- net +3V3: track 30.8 -> 50.1 mm
- net +12V: track 315.5 -> 327.3 mm, vias 1 -> 2
- net /Controller/ADC3V3: track 0.00 -> 7.99 mm
- net Net-(D30-Pad2): track 0.00 -> 1.82 mm
- net Net-(D19-Pad2): track 0.00 -> 1.82 mm
